Commit message: Fix joint direction

File: kuroko_description/xacro/kuroko/parts/arm_l.xacro (robot description, xacro)
@@ -55,5 +55,5 @@
       <child link="elbow_l_front_link"/>
       <origin xyz="0 -0.023 -0.036" rpy="0 0 0"/>
-      <axis xyz="0 -1 0"/>
+      <axis xyz="0 1 0"/>
       <limit effort="3.1" lower="-2.6180" upper="2.6180" velocity="6.5"/>
       <dynamics damping="0.477" friction="0.0"/>

File: kuroko_description/xacro/kuroko/parts/arm_r.xacro (robot description, xacro)
@@ -7,5 +7,5 @@
       <child link="shoulder_r_pitch_link"/>
       <origin xyz="0 -0.128 0.01275" rpy="0 0 0"/>
-      <axis xyz="0 -1 0"/>
+      <axis xyz="0 1 0"/>
       <limit effort="3.1" lower="-3.14" upper="3.14" velocity="6.5"/>
       <dynamics damping="0.477" friction="0.0"/>
@@ -81,5 +81,5 @@
       <child link="elbow_r_rear_link"/>
       <origin xyz="0 0.024 -0.036" rpy="0 0 0"/>
-      <axis xyz="0 -1 0"/>
+      <axis xyz="0 1 0"/>
       <limit effort="3.1" lower="-2.6180" upper="2.6180" velocity="6.5"/>
       <dynamics damping="0.477" friction="0.0"/>
