Commit message: Toe collision into spheres

File: kuroko_description/xacro/kuroko/parts/leg_l.xacro (robot description, xacro)
@@ -376,6 +376,34 @@
         <xacro:box_visual xyz="0 0 -0.004" rpy="0 0 0" size="0.12 0.075 0.008"/>
       </xacro:if>
-      <xacro:box_collision xyz="0 0 -0.004" rpy="0 0 0" size="0.12 0.075 0.008"/>
       <xacro:box_inertial xyz="0 0 -0.004" rpy="0 0 0" size="0.12 0.075 0.008" mass="0.043"/>
+      <!-- <xacro:box_collision xyz="0 0 -0.004" rpy="0 0 0" size="0.12 0.075 0.008"/> -->
+      <collision>
+        <origin xyz="0.052 0.0295 0" rpy="0 0 0" />
+        <geometry>
+          <sphere radius="0.008" />
+        </geometry>
+        <material name="gray" />
+      </collision>
+      <collision>
+        <origin xyz="-0.052 0.0295 0" rpy="0 0 0" />
+        <geometry>
+          <sphere radius="0.008" />
+        </geometry>
+        <material name="gray" />
+      </collision>
+      <collision>
+        <origin xyz="-0.052 -0.0295 0" rpy="0 0 0" />
+        <geometry>
+          <sphere radius="0.008" />
+        </geometry>
+        <material name="gray" />
+      </collision>
+      <collision>
+        <origin xyz="0.052 -0.0295 0" rpy="0 0 0" />
+        <geometry>
+          <sphere radius="0.008" />
+        </geometry>
+        <material name="gray" />
+      </collision>
     </link>
   </xacro:macro>

File: kuroko_description/xacro/kuroko/parts/leg_r.xacro (robot description, xacro)
@@ -377,6 +377,34 @@
         <xacro:box_visual xyz="0 0 -0.004" rpy="0 0 0" size="0.12 0.075 0.008"/>
       </xacro:if>
-      <xacro:box_collision xyz="0 0 -0.004" rpy="0 0 0" size="0.12 0.075 0.008"/>
       <xacro:box_inertial xyz="0 0 -0.004" rpy="0 0 0" size="0.12 0.075 0.008" mass="0.043"/>
+      <!-- <xacro:box_collision xyz="0 0 -0.004" rpy="0 0 0" size="0.12 0.075 0.008"/> -->
+      <collision>
+        <origin xyz="0.052 0.0295 0" rpy="0 0 0" />
+        <geometry>
+          <sphere radius="0.008" />
+        </geometry>
+        <material name="gray" />
+      </collision>
+      <collision>
+        <origin xyz="-0.052 0.0295 0" rpy="0 0 0" />
+        <geometry>
+          <sphere radius="0.008" />
+        </geometry>
+        <material name="gray" />
+      </collision>
+      <collision>
+        <origin xyz="-0.052 -0.0295 0" rpy="0 0 0" />
+        <geometry>
+          <sphere radius="0.008" />
+        </geometry>
+        <material name="gray" />
+      </collision>
+      <collision>
+        <origin xyz="0.052 -0.0295 0" rpy="0 0 0" />
+        <geometry>
+          <sphere radius="0.008" />
+        </geometry>
+        <material name="gray" />
+      </collision>
     </link>
   </xacro:macro>

Commit message: Fix joint direction

File: kuroko_description/xacro/kuroko/parts/leg_l.xacro (robot description, xacro)
@@ -7,6 +7,6 @@
       <child link="hip_l_roll_link"/>
       <origin xyz="0 0 -0.08425" rpy="0 0 0"/>
-      <axis xyz="-1 0 0"/>
-      <limit effort="3.1" lower="-0.5550" upper="1.8640" velocity="6.5"/>
+      <axis xyz="1 0 0"/>
+      <limit effort="3.1" lower="-1.8640" upper="0.5550" velocity="6.5"/>
       <dynamics damping="0.477" friction="0.0"/>
     </joint>
@@ -57,6 +57,6 @@
       <child link="shin_l_active_link"/>
       <origin xyz="-0.0185 0.02925 -0.0305" rpy="0 1.047197551 0"/>
-      <axis xyz="0 -1 0"/>
-      <limit effort="8.9" lower="-0.4974" upper="1.8588" velocity="6.9"/>
+      <axis xyz="0 1 0"/>
+      <limit effort="8.9" lower="-1.8588" upper="0.4974" velocity="6.9"/>
       <dynamics damping="1.29" friction="0.0"/>
     </joint>
@@ -359,5 +359,5 @@
       <child link="ankle_l_yaw_link"/>
       <origin xyz="0 0 -0.03825" rpy="0 0 0"/>
-      <axis xyz="0 0 -1"/>
+      <axis xyz="0 0 1"/>
       <limit effort="3.1" lower="-3.1416" upper="3.1416" velocity="6.5"/>
       <dynamics damping="0.477" friction="0.0"/>

File: kuroko_description/xacro/kuroko/parts/leg_r.xacro (robot description, xacro)
@@ -32,5 +32,5 @@
       <child link="hip_r_pitch_link"/>
       <origin xyz="0 -0.027 0" rpy="0 0 0"/>
-      <axis xyz="0 -1 0"/>
+      <axis xyz="0 1 0"/>
       <limit effort="3.1" lower="-3.1" upper="3.1" velocity="6.5"/>
       <dynamics damping="0.477" friction="0.0"/>
@@ -360,5 +360,5 @@
       <child link="ankle_r_yaw_link"/>
       <origin xyz="0 0 -0.03825" rpy="0 0 0"/>
-      <axis xyz="0 0 -1"/>
+      <axis xyz="0 0 1"/>
       <limit effort="3.1" lower="-3.1" upper="3.1" velocity="6.5"/>
       <dynamics damping="0.477" friction="0.0"/>

Commit message: Fix joint direction

File: kuroko_description/xacro/kuroko/parts/leg_l.xacro (robot description, xacro)
@@ -82,6 +82,6 @@
       <child link="thigh_l_active_link"/>
       <origin xyz="0.015 0.02925 -0.0305" rpy="0 -0.785398163 0"/>
-      <axis xyz="0 -1 0"/>
-      <limit effort="8.9" lower="-1.8588" upper="0.4974" velocity="6.9"/>
+      <axis xyz="0 1 0"/>
+      <limit effort="8.9" lower="-0.4974" upper="1.8588" velocity="6.9"/>
       <dynamics damping="1.29" friction="0.0"/>
     </joint>
@@ -110,5 +110,5 @@
         <limit effort="0" lower="-3.1416" upper="3.1416" velocity="1000"/>
         <dynamics damping="0.0" friction="0.0"/>
-        <mimic joint="thigh_l_active" multiplier="1" offset="0"/>
+        <mimic joint="thigh_l_active" multiplier="-1" offset="0"/>
       </joint>
       <link name="shin_l_front_mimic_link"/>
@@ -120,5 +120,5 @@
         <limit effort="0" lower="-3.1416" upper="3.1416" velocity="1000"/>
         <dynamics damping="0.0" friction="0.0"/>
-        <mimic joint="shin_l_active" multiplier="-1" offset="0"/>
+        <mimic joint="shin_l_active" multiplier="1" offset="0"/>
       </joint>
     </xacro:unless>
@@ -154,7 +154,7 @@
       <origin xyz="-0.0185 0.02925 -0.0305" rpy="0 -0.785398163 0"/>
       <axis xyz="0 1 0"/>
-      <limit effort="0" lower="-0.4974" upper="1.8588" velocity="1000"/>
+      <limit effort="0" lower="-3.1416" upper="3.1416" velocity="1000"/>
       <dynamics damping="0" friction="0"/>
-      <mimic joint="thigh_l_active" multiplier="-1" offset="0"/>
+      <mimic joint="thigh_l_active" multiplier="1" offset="0"/>
     </joint>
     <link name="thigh_l_middle_passive_link">
@@ -182,5 +182,5 @@
         <limit effort="0" lower="-3.1416" upper="3.1416" velocity="1000"/>
         <dynamics damping="0.0" friction="0.0"/>
-        <mimic joint="thigh_l_active" multiplier="1" offset="0"/>
+        <mimic joint="thigh_l_active" multiplier="-1" offset="0"/>
       </joint>
       <link name="shin_l_rear_mimic_link"/>
@@ -192,5 +192,5 @@
         <limit effort="0" lower="-3.1416" upper="3.1416" velocity="1000"/>
         <dynamics damping="0.0" friction="0.0"/>
-        <mimic joint="shin_l_active" multiplier="-1" offset="0"/>
+        <mimic joint="shin_l_active" multiplier="1" offset="0"/>
       </joint>
     </xacro:unless>
@@ -226,7 +226,7 @@
       <origin xyz="0 0 0" rpy="0 -0.785398164 0"/>
       <axis xyz="0 1 0"/>
-      <limit effort="0" lower="-3.141592654" upper="3.141592654" velocity="1000.0"/>
+      <limit effort="0" lower="-3.1416" upper="3.1416" velocity="1000.0"/>
       <dynamics damping="0.0" friction="0.0"/>
-      <mimic joint="shin_l_active" multiplier="1" offset="0"/>
+      <mimic joint="shin_l_active" multiplier="-1" offset="0"/>
     </joint>
     <link name="knee_l_passive_link">
@@ -258,5 +258,5 @@
         <limit effort="0" lower="-3.1416" upper="3.1416" velocity="1000"/>
         <dynamics damping="0.0" friction="0.0"/>
-        <mimic joint="thigh_l_active" multiplier="-1" offset="0"/>
+        <mimic joint="thigh_l_active" multiplier="1" offset="0"/>
       </joint>
       <link name="thigh_l_rear_mimic_link"/>
@@ -268,5 +268,5 @@
         <limit effort="0" lower="-3.1416" upper="3.1416" velocity="1000"/>
         <dynamics damping="0.0" friction="0.0"/>
-        <mimic joint="shin_l_active" multiplier="1" offset="0"/>
+        <mimic joint="shin_l_active" multiplier="-1" offset="0"/>
       </joint>
     </xacro:unless>
@@ -306,7 +306,7 @@
       <origin xyz="0 0 -0.1" rpy="0 -0.785398163 0"/>
       <axis xyz="0 1 0"/>
-      <limit effort="0" lower="-0.4974" upper="1.8588" velocity="1000.0"/>
+      <limit effort="0" lower="-3.1416" upper="3.1416" velocity="1000.0"/>
       <dynamics damping="0.0" friction="0.0"/>
-      <mimic joint="shin_l_active" multiplier="1" offset="0"/>
+      <mimic joint="shin_l_active" multiplier="-1" offset="0"/>
     </joint>
     <link name="ankle_l_rear_passive_link">

File: kuroko_description/xacro/kuroko/parts/leg_r.xacro (robot description, xacro)
@@ -154,5 +154,5 @@
       <origin xyz="-0.0185 -0.02925 -0.0305" rpy="0 -0.785398163 0"/>
       <axis xyz="0 1 0"/>
-      <limit effort="0" lower="-0.4974" upper="1.8588" velocity="1000"/>
+      <limit effort="0" lower="-3.1416" upper="3.1416" velocity="1000"/>
       <dynamics damping="0" friction="0"/>
       <mimic joint="thigh_r_active" multiplier="1" offset="0"/>
@@ -226,5 +226,5 @@
       <origin xyz="0 0 0" rpy="0 -0.785398164 0"/>
       <axis xyz="0 1 0"/>
-      <limit effort="0" lower="-3.141592654" upper="3.141592654" velocity="1000.0"/>
+      <limit effort="0" lower="-3.1416" upper="3.1416" velocity="1000.0"/>
       <dynamics damping="0.0" friction="0.0"/>
       <mimic joint="shin_r_active" multiplier="-1" offset="0"/>
@@ -306,5 +306,5 @@
       <origin xyz="0 0 -0.1" rpy="0 -0.785398163 0"/>
       <axis xyz="0 1 0"/>
-      <limit effort="0" lower="-0.4974" upper="1.8588" velocity="1000.0"/>
+      <limit effort="0" lower="-3.1416" upper="3.1416" velocity="1000.0"/>
       <dynamics damping="0.0" friction="0.0"/>
       <mimic joint="shin_r_active" multiplier="-1" offset="0"/>

Commit message: Fix xacro

File: kuroko_description/xacro/kuroko/parts/leg_l.xacro (robot description, xacro)
@@ -108,5 +108,5 @@
         <origin xyz="0 0 -0.1" rpy="0 0.785398163 0"/>
         <axis xyz="0 1 0"/>
-        <limit effort="0" lower="-3.1416" upper="3.1416" velocity="1000"/>
+        <limit effort="0" lower="-1.8588" upper="0.4974" velocity="1000"/>
         <dynamics damping="0.0" friction="0.0"/>
         <mimic joint="thigh_l_active" multiplier="-1" offset="0"/>
@@ -118,5 +118,5 @@
         <origin xyz="0 0 0" rpy="0 0.785398163 0"/>
         <axis xyz="0 1 0"/>
-        <limit effort="0" lower="-3.1416" upper="3.1416" velocity="1000"/>
+        <limit effort="0" lower="-1.8588" upper="0.4974" velocity="1000"/>
         <dynamics damping="0.0" friction="0.0"/>
         <mimic joint="shin_l_active" multiplier="1" offset="0"/>
@@ -154,5 +154,5 @@
       <origin xyz="-0.0185 0.02925 -0.0305" rpy="0 -0.785398163 0"/>
       <axis xyz="0 1 0"/>
-      <limit effort="0" lower="-3.1416" upper="3.1416" velocity="1000"/>
+      <limit effort="0" lower="-0.4974" upper="1.8588" velocity="1000"/>
       <dynamics damping="0" friction="0"/>
       <mimic joint="thigh_l_active" multiplier="1" offset="0"/>
@@ -180,5 +180,5 @@
         <origin xyz="0 0 -0.1" rpy="0 0.785398163 0"/>
         <axis xyz="0 1 0"/>
-        <limit effort="0" lower="-3.1416" upper="3.1416" velocity="1000"/>
+        <limit effort="0" lower="-1.8588" upper="0.4974" velocity="1000"/>
         <dynamics damping="0.0" friction="0.0"/>
         <mimic joint="thigh_l_active" multiplier="-1" offset="0"/>
@@ -190,5 +190,5 @@
         <origin xyz="0 0 0" rpy="0 0.785398163 0"/>
         <axis xyz="0 1 0"/>
-        <limit effort="0" lower="-3.1416" upper="3.1416" velocity="1000"/>
+        <limit effort="0" lower="-1.8588" upper="0.4974" velocity="1000"/>
         <dynamics damping="0.0" friction="0.0"/>
         <mimic joint="shin_l_active" multiplier="1" offset="0"/>
@@ -226,5 +226,5 @@
       <origin xyz="0 0 0" rpy="0 -0.785398164 0"/>
       <axis xyz="0 1 0"/>
-      <limit effort="0" lower="-3.1416" upper="3.1416" velocity="1000.0"/>
+      <limit effort="0" lower="-0.4974" upper="1.8588" velocity="1000.0"/>
       <dynamics damping="0.0" friction="0.0"/>
       <mimic joint="shin_l_active" multiplier="-1" offset="0"/>
@@ -256,5 +256,5 @@
         <origin xyz="-0.00776457 0 -0.0289778" rpy="0 -0.785398163 0"/>
         <axis xyz="0 1 0"/>
-        <limit effort="0" lower="-3.1416" upper="3.1416" velocity="1000"/>
+        <limit effort="0" lower="-0.4974" upper="1.8588" velocity="1000"/>
         <dynamics damping="0.0" friction="0.0"/>
         <mimic joint="thigh_l_active" multiplier="1" offset="0"/>
@@ -266,5 +266,5 @@
         <origin xyz="0 0 0" rpy="0 -0.785398163 0"/>
         <axis xyz="0 1 0"/>
-        <limit effort="0" lower="-3.1416" upper="3.1416" velocity="1000"/>
+        <limit effort="0" lower="-0.4974" upper="1.8588" velocity="1000"/>
         <dynamics damping="0.0" friction="0.0"/>
         <mimic joint="shin_l_active" multiplier="-1" offset="0"/>
@@ -306,5 +306,5 @@
       <origin xyz="0 0 -0.1" rpy="0 -0.785398163 0"/>
       <axis xyz="0 1 0"/>
-      <limit effort="0" lower="-3.1416" upper="3.1416" velocity="1000.0"/>
+      <limit effort="0" lower="-0.4974" upper="1.8588" velocity="1000.0"/>
       <dynamics damping="0.0" friction="0.0"/>
       <mimic joint="shin_l_active" multiplier="-1" offset="0"/>

File: kuroko_description/xacro/kuroko/parts/leg_r.xacro (robot description, xacro)
@@ -108,5 +108,5 @@
         <origin xyz="0 0 -0.1" rpy="0 0.785398163 0"/>
         <axis xyz="0 1 0"/>
-        <limit effort="0" lower="-3.1416" upper="3.1416" velocity="1000"/>
+        <limit effort="0" lower="-1.8588" upper="0.4974" velocity="1000"/>
         <dynamics damping="0.0" friction="0.0"/>
         <mimic joint="thigh_r_active" multiplier="-1" offset="0"/>
@@ -118,5 +118,5 @@
         <origin xyz="0 0 0" rpy="0 0.785398163 0"/>
         <axis xyz="0 1 0"/>
-        <limit effort="0" lower="-3.1416" upper="3.1416" velocity="1000"/>
+        <limit effort="0" lower="-1.8588" upper="0.4974" velocity="1000"/>
         <dynamics damping="0.0" friction="0.0"/>
         <mimic joint="shin_r_active" multiplier="1" offset="0"/>
@@ -154,5 +154,5 @@
       <origin xyz="-0.0185 -0.02925 -0.0305" rpy="0 -0.785398163 0"/>
       <axis xyz="0 1 0"/>
-      <limit effort="0" lower="-3.1416" upper="3.1416" velocity="1000"/>
+      <limit effort="0" lower="-0.4974" upper="1.8588" velocity="1000"/>
       <dynamics damping="0" friction="0"/>
       <mimic joint="thigh_r_active" multiplier="1" offset="0"/>
@@ -180,5 +180,5 @@
         <origin xyz="0 0 -0.1" rpy="0 0.785398163 0"/>
         <axis xyz="0 1 0"/>
-        <limit effort="0" lower="-3.1416" upper="3.1416" velocity="1000"/>
+        <limit effort="0" lower="-1.8588" upper="0.4974" velocity="1000"/>
         <dynamics damping="0.0" friction="0.0"/>
         <mimic joint="thigh_r_active" multiplier="-1" offset="0"/>
@@ -190,5 +190,5 @@
         <origin xyz="0 0 0" rpy="0 0.785398163 0"/>
         <axis xyz="0 1 0"/>
-        <limit effort="0" lower="-3.1416" upper="3.1416" velocity="1000"/>
+        <limit effort="0" lower="-1.8588" upper="0.4974" velocity="1000"/>
         <dynamics damping="0.0" friction="0.0"/>
         <mimic joint="shin_r_active" multiplier="1" offset="0"/>
@@ -226,5 +226,5 @@
       <origin xyz="0 0 0" rpy="0 -0.785398164 0"/>
       <axis xyz="0 1 0"/>
-      <limit effort="0" lower="-3.1416" upper="3.1416" velocity="1000.0"/>
+      <limit effort="0" lower="-0.4974" upper="1.8588" velocity="1000.0"/>
       <dynamics damping="0.0" friction="0.0"/>
       <mimic joint="shin_r_active" multiplier="-1" offset="0"/>
@@ -256,5 +256,5 @@
         <origin xyz="-0.00776457 0 -0.0289778" rpy="0 -0.785398163 0"/>
         <axis xyz="0 1 0"/>
-        <limit effort="0" lower="-3.1416" upper="3.1416" velocity="1000"/>
+        <limit effort="0" lower="-0.4974" upper="1.8588" velocity="1000"/>
         <dynamics damping="0.0" friction="0.0"/>
         <mimic joint="thigh_r_active" multiplier="1" offset="0"/>
@@ -266,5 +266,5 @@
         <origin xyz="0 0 0" rpy="0 -0.785398163 0"/>
         <axis xyz="0 1 0"/>
-        <limit effort="0" lower="-3.1416" upper="3.1416" velocity="1000"/>
+        <limit effort="0" lower="-0.4974" upper="1.8588" velocity="1000"/>
         <dynamics damping="0.0" friction="0.0"/>
         <mimic joint="shin_r_active" multiplier="-1" offset="0"/>
@@ -306,5 +306,5 @@
       <origin xyz="0 0 -0.1" rpy="0 -0.785398163 0"/>
       <axis xyz="0 1 0"/>
-      <limit effort="0" lower="-3.1416" upper="3.1416" velocity="1000.0"/>
+      <limit effort="0" lower="-0.4974" upper="1.8588" velocity="1000.0"/>
       <dynamics damping="0.0" friction="0.0"/>
       <mimic joint="shin_r_active" multiplier="-1" offset="0"/>

Commit message: Add robot_name arg

File: kuroko_description/xacro/kuroko/parts/leg_l.xacro (robot description, xacro)
@@ -1,5 +1,5 @@
 <?xml version="1.0"?>
 <robot xmlns:xacro="http://www.ros.org/wiki/xacro">
-  <xacro:macro name="leg_l_xacro" params="gazebo:=false box_visual:=false">
+  <xacro:macro name="leg_l_xacro" params="gazebo:=false box_visual:=false robot_name:=kuroko">
     <!-- Link conencts from body. Hip first. -->
     <joint name="hip_l_roll" type="revolute">
@@ -379,30 +379,30 @@
       <!-- <xacro:box_collision xyz="0 0 -0.004" rpy="0 0 0" size="0.12 0.075 0.008"/> -->
       <collision>
-        <origin xyz="0.052 0.0295 0" rpy="0 0 0" />
+        <origin xyz="0.052 0.0295 0" rpy="0 0 0"/>
         <geometry>
-          <sphere radius="0.008" />
+          <sphere radius="0.008"/>
         </geometry>
-        <material name="gray" />
+        <material name="gray"/>
       </collision>
       <collision>
-        <origin xyz="-0.052 0.0295 0" rpy="0 0 0" />
+        <origin xyz="-0.052 0.0295 0" rpy="0 0 0"/>
         <geometry>
-          <sphere radius="0.008" />
+          <sphere radius="0.008"/>
         </geometry>
-        <material name="gray" />
+        <material name="gray"/>
       </collision>
       <collision>
-        <origin xyz="-0.052 -0.0295 0" rpy="0 0 0" />
+        <origin xyz="-0.052 -0.0295 0" rpy="0 0 0"/>
         <geometry>
-          <sphere radius="0.008" />
+          <sphere radius="0.008"/>
         </geometry>
-        <material name="gray" />
+        <material name="gray"/>
       </collision>
       <collision>
-        <origin xyz="0.052 -0.0295 0" rpy="0 0 0" />
+        <origin xyz="0.052 -0.0295 0" rpy="0 0 0"/>
         <geometry>
-          <sphere radius="0.008" />
+          <sphere radius="0.008"/>
         </geometry>
-        <material name="gray" />
+        <material name="gray"/>
       </collision>
     </link>

File: kuroko_description/xacro/kuroko/parts/leg_r.xacro (robot description, xacro)
@@ -1,5 +1,5 @@
 <?xml version="1.0"?>
 <robot xmlns:xacro="http://www.ros.org/wiki/xacro">
-  <xacro:macro name="leg_r_xacro" params="gazebo:=false box_visual:=false">
+  <xacro:macro name="leg_r_xacro" params="gazebo:=false box_visual:=false robot_name:=kuroko">
     <!-- Link conencts from body. Hip first. -->
     <joint name="hip_r_roll" type="revolute">
@@ -380,30 +380,30 @@
       <!-- <xacro:box_collision xyz="0 0 -0.004" rpy="0 0 0" size="0.12 0.075 0.008"/> -->
       <collision>
-        <origin xyz="0.052 0.0295 0" rpy="0 0 0" />
+        <origin xyz="0.052 0.0295 0" rpy="0 0 0"/>
         <geometry>
-          <sphere radius="0.008" />
+          <sphere radius="0.008"/>
         </geometry>
-        <material name="gray" />
+        <material name="gray"/>
       </collision>
       <collision>
-        <origin xyz="-0.052 0.0295 0" rpy="0 0 0" />
+        <origin xyz="-0.052 0.0295 0" rpy="0 0 0"/>
         <geometry>
-          <sphere radius="0.008" />
+          <sphere radius="0.008"/>
         </geometry>
-        <material name="gray" />
+        <material name="gray"/>
       </collision>
       <collision>
-        <origin xyz="-0.052 -0.0295 0" rpy="0 0 0" />
+        <origin xyz="-0.052 -0.0295 0" rpy="0 0 0"/>
         <geometry>
-          <sphere radius="0.008" />
+          <sphere radius="0.008"/>
         </geometry>
-        <material name="gray" />
+        <material name="gray"/>
       </collision>
       <collision>
-        <origin xyz="0.052 -0.0295 0" rpy="0 0 0" />
+        <origin xyz="0.052 -0.0295 0" rpy="0 0 0"/>
         <geometry>
-          <sphere radius="0.008" />
+          <sphere radius="0.008"/>
         </geometry>
-        <material name="gray" />
+        <material name="gray"/>
       </collision>
     </link>
