Commit message: Set PID gain from yaml

File: kuroko_description/xacro/kuroko/ros2_control/gz_sim_pid_position_control.xacro (robot description, xacro)
@@ -10,9 +10,11 @@
   <!-- Controller YAML file used by gz_ros2_control::GazeboSimROS2ControlPlugin -->
   <xacro:property name="ctrl_yaml"
-                  value="$(find kuroko_description)/config/gz_position_controller.yaml" />
+    value="$(find kuroko_description)/config/gz_position_controller.yaml"/>
   <!-- Default PID parameters (can be overridden before calling the macro) -->
-  <xacro:property name="pid_kp" value="0.0" />
-  <xacro:property name="pid_ki" value="0.0" />
-  <xacro:property name="pid_kd" value="0.0" />
+  <xacro:property name="pid_kp" value="0.0"/>
+  <xacro:property name="pid_ki" value="0.0"/>
+  <xacro:property name="pid_kd" value="0.0"/>
+  <!-- Optional per-joint gain YAML (empty disables overrides) -->
+  <xacro:property name="pid_gains_yaml" value="$(find kuroko_description)/config/gz_pid_gains.yaml"/>
   <!--
     use_joint_damping:
@@ -21,5 +23,5 @@
       false -> Mode 2: do not overwrite Gazebo damping; use internal speed-dependent torque limits.
   -->
-  <xacro:property name="use_joint_damping" value="false" />
+  <xacro:property name="use_joint_damping" value="false"/>
   <!--
     release_speed_limit:
@@ -28,13 +30,16 @@
       false -> keep SDF max velocity limit as-is.
   -->
-  <xacro:property name="release_speed_limit" value="false" />
+  <xacro:property name="release_speed_limit" value="false"/>
   <!-- Load controller YAML -->
   <xacro:property name="ctrl_cfg"
-                  value="${xacro.load_yaml(ctrl_yaml)}" />
+    value="${xacro.load_yaml(ctrl_yaml)}"/>
   <!-- Extract joints list from YAML -->
   <xacro:property name="pos_joints"
-                  value="${ctrl_cfg['joint_group_position_controller']['ros__parameters']['joints']}" />
-  <!-- One ros2_control <joint> block -->
-  <xacro:macro name="gz_pid_joint_hardware_interface" params="joint_name">
+    value="${ctrl_cfg['joint_group_position_controller']['ros__parameters']['joints']}"/>
+  <!-- Load per-joint PID gain YAML if provided -->
+  <xacro:property name="pid_cfg"
+    value="${xacro.load_yaml(pid_gains_yaml) if pid_gains_yaml != '' else dict()}"/>
+  <!-- One ros2_control <joint> block (explicit gain args) -->
+  <xacro:macro name="gz_pid_joint_hardware_interface" params="joint_name kp ki kd">
     <joint name="${joint_name}">
       <!-- Commands -->
@@ -47,20 +52,31 @@
       <state_interface name="effort"/>
       <!-- Per-joint parameters consumed by gz_ros2_pid_control -->
-      <param name="kp">${pid_kp}</param>
-      <param name="ki">${pid_ki}</param>
-      <param name="kd">${pid_kd}</param>
+      <param name="kp">${kp}</param>
+      <param name="ki">${ki}</param>
+      <param name="kd">${kd}</param>
       <param name="use_joint_damping">${use_joint_damping}</param>
       <param name="release_speed_limit">${release_speed_limit}</param>
     </joint>
   </xacro:macro>
+  <!-- Recursive loop (xacro:for is not available in some environments) -->
+  <xacro:macro name="gz_pid_joint_hardware_interface_loop" params="joints">
+    <xacro:if value="${len(joints) > 0}">
+      <!-- Read per-joint overrides from pid_gains_yaml (p/i/d) -->
+      <xacro:property name="jn" value="${joints[0]}"/>
+      <xacro:property name="jg" value="${pid_cfg.get('gains', dict()).get(jn, dict())}"/>
+      <xacro:property name="jkp" value="${pid_cfg.get('gains', dict()).get(jn, dict()).get('p', pid_kp)}"/>
+      <xacro:property name="jki" value="${pid_cfg.get('gains', dict()).get(jn, dict()).get('i', pid_ki)}"/>
+      <xacro:property name="jkd" value="${pid_cfg.get('gains', dict()).get(jn, dict()).get('d', pid_kd)}"/>
+      <xacro:gz_pid_joint_hardware_interface joint_name="${jn}" kp="${jkp}" ki="${jki}" kd="${jkd}"/>
+      <xacro:gz_pid_joint_hardware_interface_loop joints="${joints[1:]}"/>
+    </xacro:if>
+  </xacro:macro>
   <!-- ros2_control hardware interface (uses the PID hardware plugin) -->
   <xacro:macro name="set_hardware_interface">
-    <ros2_control name="GazeboSimSystem" type="system">
+    <ros2_control name="GazeboSystem" type="system">
       <hardware>
         <plugin>gz_ros2_pid_control/GazeboSimPIDSystem</plugin>
       </hardware>
-      <xacro:for each="jn" value="${pos_joints}">
-        <xacro:gz_pid_joint_hardware_interface joint_name="${jn}"/>
-      </xacro:for>
+      <xacro:gz_pid_joint_hardware_interface_loop joints="${pos_joints}"/>
     </ros2_control>
   </xacro:macro>

Commit message: gains -> pid_gains

File: kuroko_description/xacro/kuroko/ros2_control/gz_sim_pid_position_control.xacro (robot description, xacro)
@@ -64,8 +64,8 @@
       <!-- Read per-joint overrides from pid_gains_yaml (p/i/d) -->
       <xacro:property name="jn" value="${joints[0]}"/>
-      <xacro:property name="jg" value="${pid_cfg.get('gains', dict()).get(jn, dict())}"/>
-      <xacro:property name="jkp" value="${pid_cfg.get('gains', dict()).get(jn, dict()).get('p', pid_kp)}"/>
-      <xacro:property name="jki" value="${pid_cfg.get('gains', dict()).get(jn, dict()).get('i', pid_ki)}"/>
-      <xacro:property name="jkd" value="${pid_cfg.get('gains', dict()).get(jn, dict()).get('d', pid_kd)}"/>
+      <xacro:property name="jg" value="${pid_cfg.get('pid_gains', dict()).get(jn, dict())}"/>
+      <xacro:property name="jkp" value="${pid_cfg.get('pid_gains', dict()).get(jn, dict()).get('p', pid_kp)}"/>
+      <xacro:property name="jki" value="${pid_cfg.get('pid_gains', dict()).get(jn, dict()).get('i', pid_ki)}"/>
+      <xacro:property name="jkd" value="${pid_cfg.get('pid_gains', dict()).get(jn, dict()).get('d', pid_kd)}"/>
       <xacro:gz_pid_joint_hardware_interface joint_name="${jn}" kp="${jkp}" ki="${jki}" kd="${jkd}"/>
       <xacro:gz_pid_joint_hardware_interface_loop joints="${joints[1:]}"/>

File: kuroko_description/xacro/kuroko/ros2_control/gz_sim_pid_trajectory_control.xacro (robot description, xacro)
@@ -60,9 +60,9 @@
       <!-- Read per-joint overrides from pid_gains_yaml (p/i/d) -->
       <xacro:property name="jkp"
-        value="${pid_cfg.get('gains', dict()).get(jn, dict()).get('p', pid_kp)}"/>
+        value="${pid_cfg.get('pid_gains', dict()).get(jn, dict()).get('p', pid_kp)}"/>
       <xacro:property name="jki"
-        value="${pid_cfg.get('gains', dict()).get(jn, dict()).get('i', pid_ki)}"/>
+        value="${pid_cfg.get('pid_gains', dict()).get(jn, dict()).get('i', pid_ki)}"/>
       <xacro:property name="jkd"
-        value="${pid_cfg.get('gains', dict()).get(jn, dict()).get('d', pid_kd)}"/>
+        value="${pid_cfg.get('pid_gains', dict()).get(jn, dict()).get('d', pid_kd)}"/>
       <xacro:gz_pid_joint_hardware_interface
         joint_name="${jn}"
