Commit message: WIP

File: kuroko_description/xacro/gazebo/gazebo_ros2_control_plugin.xacro (robot description, xacro)
@@ -1,20 +1,39 @@
-<?xml version="1.0"?>
+<?xml version="1.0" encoding="UTF-8"?>
 <robot xmlns:xacro="http://www.ros.org/wiki/xacro">
   <!--
-    Macro: gazebo_ros2_control plugin with multiple YAML parameter files.
-    Args:
-      - enabled: true/false (typically ${gazebo})
-      - robot_param: usually "robot_description"
-      - robot_param_node: usually "robot_state_publisher"
-      - controller_manager_name: optional, default "controller_manager"
-      - yaml_files: semicolon-separated list of YAML paths
-                   e.g. "$(find kuroko_description)/config/ros2_control/controller_manager.yaml;..."
+    Gazebo Classic gazebo_ros2_control plugin helper.
+    Params:
+      - enabled: bool (typically ${gazebo})
+      - yaml_files: semicolon-separated yaml list
+      - robot_param: default robot_description
+      - robot_param_node: default robot_state_publisher
+    Notes:
+      - Avoids xacro:for (not available in some ROS 2 Humble xacro setups).
+      - Expands yaml_files into multiple <parameters> tags using recursion.
   -->
   <xacro:macro name="gazebo_ros2_control_plugin"
                params="enabled
+                       yaml_files:=''
                        robot_param:=robot_description
                        robot_param_node:=robot_state_publisher
-                       controller_manager_name:=controller_manager
-                       yaml_files:=''">
+                       debug:=false">
+    <!-- Split yaml_files -->
+    <xacro:property name="_yaml_list"
+                    value="${[s for s in yaml_files.split(';') if s.strip()]}" />
+    <!-- Debug -->
+    <xacro:if value="${enabled and debug}">
+      <xacro:message text="[gazebo_ros2_control] enabled=true"/>
+      <xacro:message text="${'[gazebo_ros2_control] yaml_files=' + (','.join(_yaml_list) if len(_yaml_list)>0 else '(empty)')}"/>
+      <xacro:if value="${len(_yaml_list) == 0}">
+        <xacro:warning text="[gazebo_ros2_control] yaml_files is empty. Plugin will not load any parameters."/>
+      </xacro:if>
+    </xacro:if>
+    <!-- Recursively emit <parameters> -->
+    <xacro:macro name="_emit_params" params="paths">
+      <xacro:if value="${len(paths) > 0}">
+        <parameters>${paths[0]}</parameters>
+        <xacro:_emit_params paths="${paths[1:]}"/>
+      </xacro:if>
+    </xacro:macro>
     <xacro:if value="${enabled}">
       <gazebo>
@@ -22,10 +41,5 @@
           <robot_param>${robot_param}</robot_param>
           <robot_param_node>${robot_param_node}</robot_param_node>
-          <!-- Optional: if you want to force the name -->
-          <!-- <controller_manager_name>${controller_manager_name}</controller_manager_name> -->
-          <!-- Expand all YAML files into multiple <parameters> tags -->
-          <xacro:for each="y" value="${[s for s in yaml_files.split(';') if s.strip()]}">
-            <parameters>${y}</parameters>
-          </xacro:for>
+          <xacro:_emit_params paths="${_yaml_list}"/>
         </plugin>
       </gazebo>

Commit message: WIP

File: kuroko_description/xacro/gazebo/gazebo_ros2_control_plugin.xacro (robot description, xacro)
@@ -1,33 +1,88 @@
 <?xml version="1.0" encoding="UTF-8"?>
 <robot xmlns:xacro="http://www.ros.org/wiki/xacro">
-  <!--
-    Gazebo Classic gazebo_ros2_control plugin helper.
-    Params:
-      - enabled: bool (typically ${gazebo})
-      - yaml_files: semicolon-separated yaml list
-      - robot_param: default robot_description
-      - robot_param_node: default robot_state_publisher
-    Notes:
-      - Avoids xacro:for (not available in some ROS 2 Humble xacro setups).
-      - Expands yaml_files into multiple <parameters> tags using recursion.
-  -->
   <xacro:macro name="gazebo_ros2_control_plugin"
                params="enabled
+                       controller:=''
                        yaml_files:=''
+                       command_interface:=''
+                       debug:=false
+                       ros2_control_name:=GazeboSystem
                        robot_param:=robot_description
-                       robot_param_node:=robot_state_publisher
-                       debug:=false">
-    <!-- Split yaml_files -->
+                       robot_param_node:=robot_state_publisher">
     <xacro:property name="_yaml_list"
                     value="${[s for s in yaml_files.split(';') if s.strip()]}" />
-    <!-- Debug -->
+    <xacro:property name="_cfg_list"
+                    value="${[xacro.load_yaml(p) for p in _yaml_list]}" />
+    <xacro:property name="_cm_candidates"
+                    value="${[
+                      cfg.get('controller_manager', {}).get('ros__parameters', {}).get(controller, None)
+                      for cfg in _cfg_list
+                      if isinstance(cfg, dict)
+                    ]}" />
+    <xacro:property name="_direct_candidates"
+                    value="${[
+                      cfg.get(controller, {}).get('ros__parameters', None)
+                      for cfg in _cfg_list
+                      if isinstance(cfg, dict)
+                    ]}" />
+    <xacro:property name="_ctrl_cfg"
+                    value="${next(
+                      (c for c in _cm_candidates if isinstance(c, dict)),
+                      next((c for c in _direct_candidates if isinstance(c, dict)), {})
+                    )}" />
+    <xacro:property name="_ctrl_type"
+                    value="${_ctrl_cfg.get('type', '') if isinstance(_ctrl_cfg, dict) else ''}" />
+    <xacro:property name="_joints"
+                    value="${_ctrl_cfg.get('joints', []) if (isinstance(_ctrl_cfg, dict) and isinstance(_ctrl_cfg.get('joints', []), list)) else []}" />
+    <xacro:property name="_cmd_ifs"
+                    value="${_ctrl_cfg.get('command_interfaces', []) if (isinstance(_ctrl_cfg, dict) and isinstance(_ctrl_cfg.get('command_interfaces', []), list)) else []}" />
+    <xacro:property name="_iface_name"
+                    value="${_ctrl_cfg.get('interface_name', '') if (isinstance(_ctrl_cfg, dict) and isinstance(_ctrl_cfg.get('interface_name', ''), str)) else ''}" />
+    <xacro:property name="_cmd_if"
+                    value="${
+                      command_interface if command_interface else
+                      (
+                        (
+                          'effort' if ('effort' in _cmd_ifs) else
+                          ('position' if ('position' in _cmd_ifs) else
+                           ('velocity' if ('velocity' in _cmd_ifs) else
+                            (_cmd_ifs[0] if len(_cmd_ifs) > 0 else 'position')
+                           )
+                          )
+                        )
+                        if len(_cmd_ifs) > 0 else
+                        (
+                          (
+                            'effort' if ('effort' in _iface_name) else
+                            ('position' if ('position' in _iface_name) else
+                             ('velocity' if ('velocity' in _iface_name) else
+                              (_iface_name if _iface_name else 'position')
+                             )
+                            )
+                          )
+                          if _iface_name else
+                          (
+                            'position' if ('JointGroupPositionController' in _ctrl_type) else
+                            ('effort' if ('JointGroupEffortController' in _ctrl_type) else
+                             'position'
+                            )
+                          )
+                        )
+                      )
+                    }" />
     <xacro:if value="${enabled and debug}">
       <xacro:message text="[gazebo_ros2_control] enabled=true"/>
+      <xacro:message text="${'[gazebo_ros2_control] controller=' + (controller if controller else '(empty)')}"/>
       <xacro:message text="${'[gazebo_ros2_control] yaml_files=' + (','.join(_yaml_list) if len(_yaml_list)>0 else '(empty)')}"/>
-      <xacro:if value="${len(_yaml_list) == 0}">
-        <xacro:warning text="[gazebo_ros2_control] yaml_files is empty. Plugin will not load any parameters."/>
+      <xacro:message text="${'[gazebo_ros2_control] type=' + (_ctrl_type if _ctrl_type else '(not found)')}"/>
+      <xacro:message text="${'[gazebo_ros2_control] command_interfaces=' + (str(_cmd_ifs) if len(_cmd_ifs)>0 else '[]')}"/>
+      <xacro:message text="${'[gazebo_ros2_control] interface_name=' + (_iface_name if _iface_name else '(none)')}"/>
+      <xacro:message text="${'[gazebo_ros2_control] resolved_command_interface=' + _cmd_if}"/>
+      <xacro:message text="${'[gazebo_ros2_control] joints_count=' + str(len(_joints))}"/>
+      <xacro:message text="${'[gazebo_ros2_control] joints_head=' + (str(_joints[:6]) if len(_joints)>0 else '[]')}"/>
+      <xacro:if value="${len(_joints) == 0}">
+        <xacro:warning text="[gazebo_ros2_control] joints list is empty (no ros2_control joints will be generated)."/>
       </xacro:if>
     </xacro:if>
-    <!-- Recursively emit <parameters> -->
     <xacro:macro name="_emit_params" params="paths">
       <xacro:if value="${len(paths) > 0}">
@@ -36,7 +91,28 @@
       </xacro:if>
     </xacro:macro>
+    <xacro:macro name="_joint_block" params="joint_name cmd_if">
+      <joint name="${joint_name}">
+        <command_interface name="${cmd_if}"/>
+        <state_interface name="position"/>
+        <state_interface name="velocity"/>
+        <state_interface name="effort"/>
+      </joint>
+    </xacro:macro>
+    <xacro:macro name="_joint_loop" params="joints cmd_if">
+      <xacro:if value="${len(joints) > 0}">
+        <xacro:_joint_block joint_name="${joints[0]}" cmd_if="${cmd_if}"/>
+        <xacro:_joint_loop joints="${joints[1:]}" cmd_if="${cmd_if}"/>
+      </xacro:if>
+    </xacro:macro>
     <xacro:if value="${enabled}">
+      <!-- This block is REQUIRED so gazebo_ros2_control can start controller_manager -->
+      <ros2_control name="${ros2_control_name}" type="system">
+        <hardware>
+          <plugin>gazebo_ros2_control/GazeboSystem</plugin>
+        </hardware>
+        <xacro:_joint_loop joints="${_joints}" cmd_if="${_cmd_if}"/>
+      </ros2_control>
       <gazebo>
-        <plugin name="gazebo_ros2_control" filename="libgazebo_ros2_control.so">
+        <plugin filename="libgazebo_ros2_control.so" name="gazebo_ros2_control">
           <robot_param>${robot_param}</robot_param>
           <robot_param_node>${robot_param_node}</robot_param_node>

Commit message: WIP

File: kuroko_description/xacro/gazebo/gazebo_ros2_control_plugin.xacro (robot description, xacro)
@@ -1,4 +1,25 @@
 <?xml version="1.0" encoding="UTF-8"?>
 <robot xmlns:xacro="http://www.ros.org/wiki/xacro">
+  <!--
+    Gazebo Classic gazebo_ros2_control helper (ROS 2 Humble / restricted xacro eval safe)
+    Safe constraints:
+      - no xacro:for
+      - no isinstance()
+      - no next()
+      - no dict literal {}  (use dict())
+      - avoid len() (use list + [default] trick)
+    Params:
+      - enabled: bool
+      - controller: controller instance name (e.g. joint_trajectory_controller)
+      - yaml_files: semicolon-separated list of YAML file paths (absolute paths strongly recommended)
+      - command_interface: optional override (position/velocity/effort); empty => infer
+      - debug: print xacro-time messages
+    YAML layouts supported:
+      A) <controller>:
+           ros__parameters: { type, joints, ... }
+      B) controller_manager:
+           ros__parameters:
+             <controller>: { type, joints, ... }
+  -->
   <xacro:macro name="gazebo_ros2_control_plugin"
                params="enabled
@@ -10,13 +31,15 @@
                        robot_param:=robot_description
                        robot_param_node:=robot_state_publisher">
+    <!-- Split YAML list -->
     <xacro:property name="_yaml_list"
                     value="${[s for s in yaml_files.split(';') if s.strip()]}" />
+    <!-- Load YAMLs -->
     <xacro:property name="_cfg_list"
                     value="${[xacro.load_yaml(p) for p in _yaml_list]}" />
+    <!-- Build candidates -->
     <xacro:property name="_cm_candidates"
                     value="${[
                       cfg.get('controller_manager', {}).get('ros__parameters', {}).get(controller, None)
                       for cfg in _cfg_list
-                      if isinstance(cfg, dict)
                     ]}" />
     <xacro:property name="_direct_candidates"
@@ -24,19 +47,22 @@
                       cfg.get(controller, {}).get('ros__parameters', None)
                       for cfg in _cfg_list
-                      if isinstance(cfg, dict)
                     ]}" />
+    <!-- Pick controller config dict without next()/len():
+         - filter out None
+         - append a default dict()
+         - take first element
+    -->
+    <xacro:property name="_ctrl_cfg_cm"
+                    value="${([c for c in _cm_candidates if c is not None] + [dict()])[0]}" />
+    <xacro:property name="_ctrl_cfg_direct"
+                    value="${([c for c in _direct_candidates if c is not None] + [dict()])[0]}" />
     <xacro:property name="_ctrl_cfg"
-                    value="${next(
-                      (c for c in _cm_candidates if isinstance(c, dict)),
-                      next((c for c in _direct_candidates if isinstance(c, dict)), {})
-                    )}" />
-    <xacro:property name="_ctrl_type"
-                    value="${_ctrl_cfg.get('type', '') if isinstance(_ctrl_cfg, dict) else ''}" />
-    <xacro:property name="_joints"
-                    value="${_ctrl_cfg.get('joints', []) if (isinstance(_ctrl_cfg, dict) and isinstance(_ctrl_cfg.get('joints', []), list)) else []}" />
-    <xacro:property name="_cmd_ifs"
-                    value="${_ctrl_cfg.get('command_interfaces', []) if (isinstance(_ctrl_cfg, dict) and isinstance(_ctrl_cfg.get('command_interfaces', []), list)) else []}" />
-    <xacro:property name="_iface_name"
-                    value="${_ctrl_cfg.get('interface_name', '') if (isinstance(_ctrl_cfg, dict) and isinstance(_ctrl_cfg.get('interface_name', ''), str)) else ''}" />
+                    value="${_ctrl_cfg_cm if _ctrl_cfg_cm else _ctrl_cfg_direct}" />
+    <!-- Extract fields -->
+    <xacro:property name="_ctrl_type" value="${_ctrl_cfg.get('type', '')}" />
+    <xacro:property name="_joints" value="${_ctrl_cfg.get('joints', [])}" />
+    <xacro:property name="_cmd_ifs" value="${_ctrl_cfg.get('command_interfaces', [])}" />
+    <xacro:property name="_iface_name" value="${_ctrl_cfg.get('interface_name', '')}" />
+    <!-- Resolve command interface (explicit > command_interfaces > interface_name > type default) -->
     <xacro:property name="_cmd_if"
                     value="${
@@ -47,9 +73,9 @@
                           ('position' if ('position' in _cmd_ifs) else
                            ('velocity' if ('velocity' in _cmd_ifs) else
-                            (_cmd_ifs[0] if len(_cmd_ifs) > 0 else 'position')
+                            (_cmd_ifs[0] if _cmd_ifs else 'position')
                            )
                           )
                         )
-                        if len(_cmd_ifs) > 0 else
+                        if _cmd_ifs else
                         (
                           (
@@ -71,24 +97,30 @@
                       )
                     }" />
+    <!-- Debug -->
     <xacro:if value="${enabled and debug}">
       <xacro:message text="[gazebo_ros2_control] enabled=true"/>
       <xacro:message text="${'[gazebo_ros2_control] controller=' + (controller if controller else '(empty)')}"/>
-      <xacro:message text="${'[gazebo_ros2_control] yaml_files=' + (','.join(_yaml_list) if len(_yaml_list)>0 else '(empty)')}"/>
+      <xacro:message text="${'[gazebo_ros2_control] yaml_files=' + (','.join(_yaml_list) if _yaml_list else '(empty)')}"/>
       <xacro:message text="${'[gazebo_ros2_control] type=' + (_ctrl_type if _ctrl_type else '(not found)')}"/>
-      <xacro:message text="${'[gazebo_ros2_control] command_interfaces=' + (str(_cmd_ifs) if len(_cmd_ifs)>0 else '[]')}"/>
+      <xacro:message text="${'[gazebo_ros2_control] command_interfaces=' + (str(_cmd_ifs) if _cmd_ifs else '[]')}"/>
       <xacro:message text="${'[gazebo_ros2_control] interface_name=' + (_iface_name if _iface_name else '(none)')}"/>
       <xacro:message text="${'[gazebo_ros2_control] resolved_command_interface=' + _cmd_if}"/>
       <xacro:message text="${'[gazebo_ros2_control] joints_count=' + str(len(_joints))}"/>
-      <xacro:message text="${'[gazebo_ros2_control] joints_head=' + (str(_joints[:6]) if len(_joints)>0 else '[]')}"/>
-      <xacro:if value="${len(_joints) == 0}">
-        <xacro:warning text="[gazebo_ros2_control] joints list is empty (no ros2_control joints will be generated)."/>
+      <xacro:message text="${'[gazebo_ros2_control] joints_head=' + (str(_joints[:6]) if _joints else '[]')}"/>
+      <xacro:if value="${not _joints}">
+        <xacro:warning text="[gazebo_ros2_control] joints list is empty. No ros2_control joints will be generated."/>
+      </xacro:if>
+      <xacro:if value="${not _yaml_list}">
+        <xacro:warning text="[gazebo_ros2_control] yaml_files is empty. Plugin will not load any parameters."/>
       </xacro:if>
     </xacro:if>
+    <!-- Emit <parameters> recursively (no xacro:for) -->
     <xacro:macro name="_emit_params" params="paths">
-      <xacro:if value="${len(paths) > 0}">
+      <xacro:if value="${paths}">
         <parameters>${paths[0]}</parameters>
         <xacro:_emit_params paths="${paths[1:]}"/>
       </xacro:if>
     </xacro:macro>
+    <!-- Emit joints recursively -->
     <xacro:macro name="_joint_block" params="joint_name cmd_if">
       <joint name="${joint_name}">
@@ -100,5 +132,5 @@
     </xacro:macro>
     <xacro:macro name="_joint_loop" params="joints cmd_if">
-      <xacro:if value="${len(joints) > 0}">
+      <xacro:if value="${joints}">
         <xacro:_joint_block joint_name="${joints[0]}" cmd_if="${cmd_if}"/>
         <xacro:_joint_loop joints="${joints[1:]}" cmd_if="${cmd_if}"/>
@@ -106,5 +138,5 @@
     </xacro:macro>
     <xacro:if value="${enabled}">
-      <!-- This block is REQUIRED so gazebo_ros2_control can start controller_manager -->
+      <!-- REQUIRED: ros2_control block for gazebo_ros2_control -->
       <ros2_control name="${ros2_control_name}" type="system">
         <hardware>
@@ -113,4 +145,5 @@
         <xacro:_joint_loop joints="${_joints}" cmd_if="${_cmd_if}"/>
       </ros2_control>
+      <!-- Gazebo Classic plugin -->
       <gazebo>
         <plugin filename="libgazebo_ros2_control.so" name="gazebo_ros2_control">

Commit message: WIP

File: kuroko_description/xacro/gazebo/gazebo_ros2_control_plugin.xacro (robot description, xacro)
@@ -8,6 +8,7 @@
                        debug:=false
                        ros2_control_name:=GazeboSystem">
+    <!-- Split YAML list (strip each element) -->
     <xacro:property name="_yaml_list"
-                    value="${[s for s in yaml_files.split(';') if s.strip()]}" />
+                    value="${[s.strip() for s in yaml_files.split(';') if s.strip()]}" />
     <xacro:property name="_cfg_list"
                     value="${[xacro.load_yaml(p) for p in _yaml_list]}" />
@@ -69,10 +70,11 @@
       <xacro:message text="${'[gazebo_ros2_control] yaml_files=' + (','.join(_yaml_list) if _yaml_list else '(empty)')}"/>
       <xacro:message text="${'[gazebo_ros2_control] type=' + (_ctrl_type if _ctrl_type else '(not found)')}"/>
-      <xacro:message text="${'[gazebo_ros2_control] command_interfaces=' + (str(_cmd_ifs) if _cmd_ifs else '[]')}"/>
-      <xacro:message text="${'[gazebo_ros2_control] interface_name=' + (_iface_name if _iface_name else '(none)')}"/>
       <xacro:message text="${'[gazebo_ros2_control] resolved_command_interface=' + _cmd_if}"/>
       <xacro:message text="${'[gazebo_ros2_control] joints_count=' + str(len(_joints))}"/>
-      <xacro:message text="${'[gazebo_ros2_control] joints_head=' + (str(_joints[:6]) if _joints else '[]')}"/>
+      <xacro:if value="${not _joints}">
+        <xacro:warning text="[gazebo_ros2_control] joints list is empty -> gazebo_ros2_control will see 0 controllable joints."/>
+      </xacro:if>
     </xacro:if>
+    <!-- Emit <parameters> recursively -->
     <xacro:macro name="_emit_params" params="paths">
       <xacro:if value="${paths}">
@@ -81,5 +83,6 @@
       </xacro:if>
     </xacro:macro>
-    <xacro:macro name="_joint_block" params="joint_name cmd_if">
+    <!-- ros2_control joint entry -->
+    <xacro:macro name="_ros2_control_joint" params="joint_name cmd_if">
       <joint name="${joint_name}">
         <command_interface name="${cmd_if}"/>
@@ -89,11 +92,27 @@
       </joint>
     </xacro:macro>
+    <!-- transmission entry (SimpleTransmission) -->
+    <xacro:macro name="_transmission" params="joint_name hw_if">
+      <transmission name="${joint_name}_trans">
+        <type>transmission_interface/SimpleTransmission</type>
+        <joint name="${joint_name}">
+          <hardwareInterface>hardware_interface/${hw_if}</hardwareInterface>
+        </joint>
+        <actuator name="${joint_name}_motor">
+          <hardwareInterface>hardware_interface/${hw_if}</hardwareInterface>
+          <mechanicalReduction>1</mechanicalReduction>
+        </actuator>
+      </transmission>
+    </xacro:macro>
+    <!-- Loop joints recursively (no xacro:for) -->
     <xacro:macro name="_joint_loop" params="joints cmd_if">
       <xacro:if value="${joints}">
-        <xacro:_joint_block joint_name="${joints[0]}" cmd_if="${cmd_if}"/>
+        <xacro:_ros2_control_joint joint_name="${joints[0]}" cmd_if="${cmd_if}"/>
+        <xacro:_transmission joint_name="${joints[0]}" hw_if="${cmd_if}"/>
         <xacro:_joint_loop joints="${joints[1:]}" cmd_if="${cmd_if}"/>
       </xacro:if>
     </xacro:macro>
     <xacro:if value="${enabled}">
+      <!-- ros2_control block -->
       <ros2_control name="${ros2_control_name}" type="system">
         <hardware>
@@ -102,4 +121,5 @@
         <xacro:_joint_loop joints="${_joints}" cmd_if="${_cmd_if}"/>
       </ros2_control>
+      <!-- Gazebo Classic plugin -->
       <gazebo>
         <plugin filename="libgazebo_ros2_control.so" name="gazebo_ros2_control">
