Commit message: WIP

File: kuroko_description/xacro/gazebo/gazebo_ros2_control_plugin.xacro (robot description, xacro)
@@ -4,27 +4,21 @@
                params="enabled
                        controller:=''
-                       yaml_files:=''
+                       controller_yaml:=''
                        command_interface:=''
                        debug:=false
                        ros2_control_name:=GazeboSystem">
-    <!-- Split YAML list (strip each element) -->
-    <xacro:property name="_yaml_list"
-                    value="${[s.strip() for s in yaml_files.split(';') if s.strip()]}" />
-    <xacro:property name="_cfg_list"
-                    value="${[xacro.load_yaml(p) for p in _yaml_list]}" />
-    <xacro:property name="_cm_candidates"
-                    value="${[
-                      cfg.get('controller_manager', dict()).get('ros__parameters', dict()).get(controller, None)
-                      for cfg in _cfg_list
-                    ]}" />
-    <xacro:property name="_direct_candidates"
-                    value="${[
-                      cfg.get(controller, dict()).get('ros__parameters', None)
-                      for cfg in _cfg_list
-                    ]}" />
+    <!-- Load YAML (single file). If empty, use empty dict. -->
+    <xacro:property name="_cfg"
+                    value="${xacro.load_yaml(controller_yaml) if controller_yaml else dict()}" />
+    <!-- Support both layouts:
+         A) <controller>.ros__parameters
+         B) controller_manager.ros__parameters.<controller>
+    -->
+    <xacro:property name="_cm_params"
+                    value="${_cfg.get('controller_manager', dict()).get('ros__parameters', dict())}" />
     <xacro:property name="_ctrl_cfg_cm"
-                    value="${([c for c in _cm_candidates if c is not None] + [dict()])[0]}" />
+                    value="${_cm_params.get(controller, dict())}" />
     <xacro:property name="_ctrl_cfg_direct"
-                    value="${([c for c in _direct_candidates if c is not None] + [dict()])[0]}" />
+                    value="${_cfg.get(controller, dict()).get('ros__parameters', dict())}" />
     <xacro:property name="_ctrl_cfg"
                     value="${_ctrl_cfg_cm if _ctrl_cfg_cm else _ctrl_cfg_direct}" />
@@ -33,54 +27,48 @@
     <xacro:property name="_cmd_ifs" value="${_ctrl_cfg.get('command_interfaces', [])}" />
     <xacro:property name="_iface_name" value="${_ctrl_cfg.get('interface_name', '')}" />
-    <xacro:property name="_cmd_if"
+    <!-- Decide command interface:
+         - If user passed command_interface (non-empty): use it
+         - Else:
+           - For ForwardCommandController family: use interface_name
+           - For JTC / Pid / others: prefer command_interfaces
+    -->
+    <xacro:property name="_is_forward"
+                    value="${('ForwardCommandController' in _ctrl_type) or ('forward_command_controller' in _ctrl_type)}" />
+    <xacro:property name="_cmd_if_from_cmd_ifs"
                     value="${
-                      command_interface if command_interface else
-                      (
-                        (
-                          'effort' if ('effort' in _cmd_ifs) else
-                          ('position' if ('position' in _cmd_ifs) else
-                           ('velocity' if ('velocity' in _cmd_ifs) else
-                            (_cmd_ifs[0] if _cmd_ifs else 'position')
-                           )
-                          )
+                      ('effort' if ('effort' in _cmd_ifs) else
+                       ('position' if ('position' in _cmd_ifs) else
+                        ('velocity' if ('velocity' in _cmd_ifs) else
+                         (_cmd_ifs[0] if _cmd_ifs else 'position')
                         )
-                        if _cmd_ifs else
-                        (
-                          (
-                            'effort' if ('effort' in _iface_name) else
-                            ('position' if ('position' in _iface_name) else
-                             ('velocity' if ('velocity' in _iface_name) else
-                              (_iface_name if _iface_name else 'position')
-                             )
-                            )
-                          )
-                          if _iface_name else
-                          (
-                            'position' if ('JointGroupPositionController' in _ctrl_type) else
-                            ('effort' if ('JointGroupEffortController' in _ctrl_type) else
-                             'position'
-                            )
-                          )
-                        )
+                       )
                       )
                     }" />
+    <xacro:property name="_cmd_if_from_iface_name"
+                    value="${
+                      ('effort' if ('effort' in _iface_name) else
+                       ('position' if ('position' in _iface_name) else
+                        ('velocity' if ('velocity' in _iface_name) else
+                         (_iface_name if _iface_name else 'position')
+                        )
+                       )
+                      )
+                    }" />
+    <xacro:property name="_cmd_if_inferred"
+                    value="${_cmd_if_from_iface_name if _is_forward else _cmd_if_from_cmd_ifs}" />
+    <xacro:property name="_cmd_if"
+                    value="${command_interface if command_interface else _cmd_if_inferred}" />
     <xacro:if value="${enabled and debug}">
       <xacro:message text="[gazebo_ros2_control] enabled=true"/>
+      <xacro:message text="${'[gazebo_ros2_control] controller_yaml=' + (controller_yaml if controller_yaml else '(empty)')}"/>
       <xacro:message text="${'[gazebo_ros2_control] controller=' + (controller if controller else '(empty)')}"/>
-      <xacro:message text="${'[gazebo_ros2_control] yaml_files=' + (','.join(_yaml_list) if _yaml_list else '(empty)')}"/>
       <xacro:message text="${'[gazebo_ros2_control] type=' + (_ctrl_type if _ctrl_type else '(not found)')}"/>
-      <xacro:message text="${'[gazebo_ros2_control] resolved_command_interface=' + _cmd_if}"/>
       <xacro:message text="${'[gazebo_ros2_control] joints_count=' + str(len(_joints))}"/>
+      <xacro:message text="${'[gazebo_ros2_control] joints_head=' + (str(_joints[:8]) if _joints else '[]')}"/>
+      <xacro:message text="${'[gazebo_ros2_control] inferred_command_interface=' + _cmd_if}"/>
       <xacro:if value="${not _joints}">
-        <xacro:warning text="[gazebo_ros2_control] joints list is empty -> gazebo_ros2_control will see 0 controllable joints."/>
+        <xacro:warning text="[gazebo_ros2_control] joints list is empty (check YAML layout / controller name / joints names)."/>
       </xacro:if>
     </xacro:if>
-    <!-- Emit <parameters> recursively -->
-    <xacro:macro name="_emit_params" params="paths">
-      <xacro:if value="${paths}">
-        <parameters>${paths[0]}</parameters>
-        <xacro:_emit_params paths="${paths[1:]}"/>
-      </xacro:if>
-    </xacro:macro>
     <!-- ros2_control joint entry -->
     <xacro:macro name="_ros2_control_joint" params="joint_name cmd_if">
@@ -105,5 +93,5 @@
       </transmission>
     </xacro:macro>
-    <!-- Loop joints recursively (no xacro:for) -->
+    <!-- Loop joints recursively -->
     <xacro:macro name="_joint_loop" params="joints cmd_if">
       <xacro:if value="${joints}">
@@ -121,8 +109,8 @@
         <xacro:_joint_loop joints="${_joints}" cmd_if="${_cmd_if}"/>
       </ros2_control>
-      <!-- Gazebo Classic plugin -->
+      <!-- Gazebo Classic plugin: single YAML -->
       <gazebo>
         <plugin filename="libgazebo_ros2_control.so" name="gazebo_ros2_control">
-          <xacro:_emit_params paths="${_yaml_list}"/>
+          <parameters>${controller_yaml}</parameters>
         </plugin>
       </gazebo>

File: kuroko_description/xacro/kuroko/kuroko.xacro (robot description, xacro)
@@ -1,39 +1,30 @@
 <?xml version="1.0"?>
 <robot name="kuroko" xmlns:xacro="http://www.ros.org/wiki/xacro">
-  <!-- Arguments -->
   <xacro:arg name="gazebo" default="false"/>
   <xacro:arg name="gz_sim" default="false"/>
+  <!-- Which controller instance name you want to use (must match YAML) -->
+  <xacro:arg name="controller" default="joint_trajectory_controller"/>
+  <!-- Optional override; if empty, plugin macro may infer from YAML -->
+  <xacro:arg name="command_interface" default="position"/>
+  <!-- Single YAML file (absolute path recommended) -->
+  <xacro:arg name="controller_yaml" default=""/>
+  <!-- Print xacro-time debug messages -->
+  <xacro:arg name="debug_control" default="false"/>
   <xacro:arg name="box_visual" default="false"/>
-  <!-- Controller selection -->
-  <xacro:arg name="controller" default="joint_trajectory_controller"/>
-  <!-- Optional explicit override; empty means infer from YAML (cmd_interfaces / interface_name / type defaults) -->
-  <xacro:arg name="command_interface" default=""/>
-  <!-- Semicolon-separated YAML list to be loaded by ros2_control plugin(s) -->
-  <xacro:arg name="controller_yaml_files"
-            default="$(find kuroko_description)/config/ros2_control/controller_manager.yaml;
-                      $(find kuroko_description)/config/ros2_control/joint_state_broadcaster.yaml;
-                      $(find kuroko_description)/config/ros2_control/joint_trajectory_controller.yaml"/>
-  <!-- Debug for xacro expansion -->
-  <xacro:arg name="debug_control" default="false"/>
-  <!-- Paths -->
-  <xacro:property name="XACRO_DIR" value="$(find kuroko_description)/xacro"/>
-  <xacro:property name="MESH_DIR" value="package://kuroko_description/meshes"/>
-  <!-- Includes: physics -->
+  <xacro:property name="XACRO_DIR" value="$(find kuroko_description)/xacro" />
+  <xacro:property name="MESH_DIR" value="package://kuroko_description/meshes" />
   <xacro:include filename="${XACRO_DIR}/physics/materials.xacro"/>
   <xacro:include filename="${XACRO_DIR}/physics/box_physics.xacro"/>
   <xacro:include filename="${XACRO_DIR}/physics/gazebo_passive_joint.xacro"/>
-  <!-- Includes: parts -->
   <xacro:include filename="${XACRO_DIR}/kuroko/parts/body.xacro"/>
+  <xacro:include filename="${XACRO_DIR}/kuroko/gazebo/body.gazebo"/>
   <xacro:include filename="${XACRO_DIR}/kuroko/parts/arm_r.xacro"/>
+  <xacro:include filename="${XACRO_DIR}/kuroko/gazebo/arm_r.gazebo"/>
   <xacro:include filename="${XACRO_DIR}/kuroko/parts/arm_l.xacro"/>
+  <xacro:include filename="${XACRO_DIR}/kuroko/gazebo/arm_l.gazebo"/>
   <xacro:include filename="${XACRO_DIR}/kuroko/parts/leg_r.xacro"/>
+  <xacro:include filename="${XACRO_DIR}/kuroko/gazebo/leg_r.gazebo"/>
   <xacro:include filename="${XACRO_DIR}/kuroko/parts/leg_l.xacro"/>
-  <!-- Includes: Gazebo Classic tags for each part -->
-  <xacro:include filename="${XACRO_DIR}/kuroko/gazebo/body.gazebo"/>
-  <xacro:include filename="${XACRO_DIR}/kuroko/gazebo/arm_r.gazebo"/>
-  <xacro:include filename="${XACRO_DIR}/kuroko/gazebo/arm_l.gazebo"/>
-  <xacro:include filename="${XACRO_DIR}/kuroko/gazebo/leg_r.gazebo"/>
   <xacro:include filename="${XACRO_DIR}/kuroko/gazebo/leg_l.gazebo"/>
-  <!-- Includes: sensors -->
   <xacro:include filename="${XACRO_DIR}/sensors/range/tfluna.xacro"/>
   <xacro:include filename="${XACRO_DIR}/sensors/imu/enable_gz_imu_plugin.xacro"/>
@@ -41,19 +32,8 @@
   <xacro:include filename="${XACRO_DIR}/sensors/camera/enable_gz_rendering_plugin.xacro"/>
   <xacro:include filename="${XACRO_DIR}/sensors/camera/usb_camera.xacro"/>
-  <!-- ros2_control plugin macros -->
+  <!-- Gazebo Classic ros2_control helper -->
   <xacro:include filename="${XACRO_DIR}/gazebo/gazebo_ros2_control_plugin.xacro"/>
-  <xacro:include filename="${XACRO_DIR}/gz/gz_ros2_control_plugin.xacro"/>
-  <!-- ====================================================================== -->
-  <!-- Macro: build the robot model                                            -->
-  <!-- ====================================================================== -->
-  <xacro:macro name="kuroko_model"
-               params="gazebo:=false
-                       gz_sim:=false
-                       box_visual:=false
-                       controller:=''
-                       controller_yaml_files:=''
-                       command_interface:=''
-                       debug_control:=false">
-    <!-- Base -->
+  <!-- Main robot model macro -->
+  <xacro:macro name="kuroko_model" params="gazebo box_visual">
     <link name="body_link"/>
     <joint name="root_joint" type="fixed">
@@ -62,19 +42,14 @@
       <origin xyz="0 0 0" rpy="0 0 0"/>
     </joint>
-    <!-- Body + limbs -->
     <xacro:body_xacro box_visual="${box_visual}"/>
+    <xacro:body_gazebo/>
     <xacro:arm_r_xacro box_visual="${box_visual}"/>
+    <xacro:arm_r_gazebo/>
     <xacro:arm_l_xacro box_visual="${box_visual}"/>
+    <xacro:arm_l_gazebo/>
     <xacro:leg_r_xacro gazebo="${gazebo}" box_visual="${box_visual}"/>
+    <xacro:leg_r_gazebo/>
     <xacro:leg_l_xacro gazebo="${gazebo}" box_visual="${box_visual}"/>
-    <!-- Gazebo Classic visuals/physics tags for parts -->
-    <xacro:if value="${gazebo}">
-      <xacro:body_gazebo/>
-      <xacro:arm_r_gazebo/>
-      <xacro:arm_l_gazebo/>
-      <xacro:leg_r_gazebo/>
-      <xacro:leg_l_gazebo/>
-    </xacro:if>
-    <!-- Sensors -->
+    <xacro:leg_l_gazebo/>
     <xacro:imu_n100mini parent="waist_link" name="imu" namespace="/kuroko/sensors/imu">
       <origin xyz="-0.04 0 -0.01" rpy="0 0 0"/>
@@ -86,30 +61,15 @@
       <origin xyz="0.07 0 -0.044" rpy="0 0 0"/>
     </xacro:tfluna>
-    <!-- Sensor plugins: Gazebo backends only -->
-    <xacro:if value="${gazebo or gz_sim}">
-      <xacro:enable_gz_rendering_plugin/>
-      <xacro:enable_gz_imu_plugin/>
-    </xacro:if>
-    <!-- ros2_control plugin injection -->
-    <!-- Gazebo Classic: expects gazebo_ros2_control_plugin macro to expand yaml_files -->
+    <xacro:enable_gz_rendering_plugin/>
+    <xacro:enable_gz_imu_plugin/>
+    <!-- ros2_control (Gazebo Classic): enabled only when gazebo:=true -->
     <xacro:gazebo_ros2_control_plugin
       enabled="${gazebo}"
-      yaml_files="${controller_yaml_files}"/>
-    <!-- Gazebo Sim: use the new gz_ros2_control_setup macro -->
-    <xacro:gz_ros2_control_setup
-      enabled="${gz_sim}"
-      controller="${controller}"
-      yaml_files="${controller_yaml_files}"
-      command_interface="${command_interface}"
-      debug="${debug_control}"/>
+      controller="$(arg controller)"
+      controller_yaml="$(arg controller_yaml)"
+      command_interface="$(arg command_interface)"
+      debug="$(arg debug_control)"/>
   </xacro:macro>
   <!-- Instantiate -->
-  <xacro:kuroko_model
-    gazebo="$(arg gazebo)"
-    gz_sim="$(arg gz_sim)"
-    box_visual="$(arg box_visual)"
-    controller="$(arg controller)"
-    controller_yaml_files="$(arg controller_yaml_files)"
-    command_interface="$(arg command_interface)"
-    debug_control="$(arg debug_control)"/>
+  <xacro:kuroko_model gazebo="$(arg gazebo)" box_visual="$(arg box_visual)"/>
 </robot>
