Commit message: WIP

File: kuroko_description/xacro/gazebo/gazebo_ros2_control_system.xacro (robot description, xacro)
@@ -8,3 +8,15 @@
     </ros2_control>
   </xacro:macro>
+  <xacro:macro name="kuroko_gazebo_ros2_control_plugin" params="controller_yaml:='' controller_manager_name:='controller_manager'">
+    <gazebo>
+      <plugin name="gazebo_ros2_control" filename="libgazebo_ros2_control.so">
+        <xacro:if value="${controller_yaml != ''}">
+          <parameters>${controller_yaml}</parameters>
+        </xacro:if>
+        <xacro:if value="${controller_manager_name != ''}">
+          <controller_manager_name>${controller_manager_name}</controller_manager_name>
+        </xacro:if>
+      </plugin>
+    </gazebo>
+  </xacro:macro>
 </robot>

File: kuroko_description/xacro/kuroko/kuroko.xacro (robot description, xacro)
@@ -4,4 +4,6 @@
   <xacro:arg name="gazebo_hardware_interface" default="position"/>
   <xacro:arg name="box_visual" default="false"/>
+  <!-- Optional ros2_control controller parameters YAML for Gazebo Classic plugin -->
+  <xacro:arg name="controller_yaml" default=""/>
   <xacro:property name="XACRO_DIR" value="$(find kuroko_description)/xacro" />
   <xacro:property name="MESH_DIR" value="$(find kuroko_description)/meshes" />
@@ -58,8 +60,8 @@
     <xacro:if value="${gazebo}">
       <xacro:if value="${gazebo_hardware_interface=='position'}">
-        <xacro:kuroko_transmission_position/>
+        <xacro:kuroko_transmission_position controller_yaml="$(arg controller_yaml)" namespace="/"/>
       </xacro:if>
       <xacro:if value="${gazebo_hardware_interface=='effort'}">
-        <xacro:kuroko_transmission_effort/>
+        <xacro:kuroko_transmission_effort controller_yaml="$(arg controller_yaml)" namespace="/"/>
       </xacro:if>
     </xacro:if>
