Commit message: WIP

File: kuroko_description/xacro/gazebo/gazebo_ros2_hardware_interface.xacro (robot description, xacro)
@@ -4,11 +4,11 @@
     Transmission generators (no YAML dependency)
     Single joint:
-      <xacro:set_effort_interface joint_name="joint1"/>
-      <xacro:set_velocity_interface joint_name="joint1"/>
-      <xacro:set_position_interface joint_name="joint1"/>
+      <xacro:set_effort_hardware_interface joint_name="joint1"/>
+      <xacro:set_velocity_hardware_interface joint_name="joint1"/>
+      <xacro:set_position_hardware_interface joint_name="joint1"/>
     Multiple joints:
-      <xacro:set_effort_interfaces joints="${['joint1','joint2']}"/>
-      <xacro:set_velocity_interfaces joints="${['joint1','joint2']}"/>
-      <xacro:set_position_interfaces joints="${['joint1','joint2']}"/>
+      <xacro:set_effort_hardware_interfaces joints="${['joint1','joint2']}"/>
+      <xacro:set_velocity_hardware_interfaces joints="${['joint1','joint2']}"/>
+      <xacro:set_position_hardware_interfaces joints="${['joint1','joint2']}"/>
   -->
   <!-- Generic transmission block -->
@@ -39,31 +39,49 @@
   </xacro:macro>
   <!-- Public: single joint -->
-  <xacro:macro name="set_effort_interface" params="joint_name">
+  <xacro:macro name="set_effort_hardware_interface" params="joint_name">
     <xacro:_effort_transmission joint_name="${joint_name}"/>
   </xacro:macro>
-  <xacro:macro name="set_velocity_interface" params="joint_name">
+  <xacro:macro name="set_velocity_hardware_interface" params="joint_name">
     <xacro:_velocity_transmission joint_name="${joint_name}"/>
   </xacro:macro>
-  <xacro:macro name="set_position_interface" params="joint_name">
+  <xacro:macro name="set_position_hardware_interface" params="joint_name">
     <xacro:_position_transmission joint_name="${joint_name}"/>
   </xacro:macro>
   <!-- Public: multiple joints (recursive inside) -->
-  <xacro:macro name="set_effort_interfaces" params="joints">
+  <xacro:macro name="set_effort_hardware_interfaces" params="joints">
     <xacro:if value="${len(joints) > 0}">
       <xacro:_effort_transmission joint_name="${joints[0]}"/>
-      <xacro:set_effort_interfaces joints="${joints[1:]}"/>
+      <xacro:set_effort_hardware_interfaces joints="${joints[1:]}"/>
     </xacro:if>
   </xacro:macro>
-  <xacro:macro name="set_velocity_interfaces" params="joints">
+  <xacro:macro name="set_velocity_hardware_interfaces" params="joints">
     <xacro:if value="${len(joints) > 0}">
       <xacro:_velocity_transmission joint_name="${joints[0]}"/>
-      <xacro:set_velocity_interfaces joints="${joints[1:]}"/>
+      <xacro:set_velocity_hardware_interfaces joints="${joints[1:]}"/>
     </xacro:if>
   </xacro:macro>
-  <xacro:macro name="set_position_interfaces" params="joints">
+  <xacro:macro name="set_position_hardware_interfaces" params="joints">
     <xacro:if value="${len(joints) > 0}">
       <xacro:_position_transmission joint_name="${joints[0]}"/>
-      <xacro:set_position_interfaces joints="${joints[1:]}"/>
+      <xacro:set_position_hardware_interfaces joints="${joints[1:]}"/>
     </xacro:if>
   </xacro:macro>
+  <xacro:macro name="gazebo_ros2_control_system">
+    <ros2_control name="GazeboSystem" type="system">
+      <hardware>
+        <plugin>gazebo_ros2_control/GazeboSystem</plugin>
+      </hardware>
+    </ros2_control>
+  </xacro:macro>
+  <xacro:macro name="gazebo_ros2_control_plugin" params="controller_yaml:=''">
+    <gazebo>
+      <plugin name="gazebo_ros2_control" filename="libgazebo_ros2_control.so">
+        <robot_param>robot_description</robot_param>
+        <robot_param_node>robot_state_publisher</robot_param_node>
+        <xacro:if value="${controller_yaml != ''}">
+          <parameters>${controller_yaml}</parameters>
+        </xacro:if>
+      </plugin>
+    </gazebo>
+  </xacro:macro>
 </robot>

File: kuroko_description/xacro/kuroko/kuroko.xacro (robot description, xacro)
@@ -27,5 +27,5 @@
   <xacro:include filename="${XACRO_DIR}/sensors/camera/usb_camera.xacro"/>
   <!-- Gazebo Classic ros2_control helper -->
-  <xacro:include filename="${XACRO_DIR}/kuroko/gazebo/kuroko_transmission.gazebo"/>
+  <xacro:include filename="${XACRO_DIR}/kuroko/gazebo/kuroko_command_interface.gazebo"/>
   <!-- Main robot model macro -->
   <xacro:macro name="kuroko_model" params="gazebo gazebo_hardware_interface box_visual">
@@ -60,8 +60,8 @@
     <xacro:if value="${gazebo}">
       <xacro:if value="${gazebo_hardware_interface=='position'}">
-        <xacro:kuroko_transmission_position controller_yaml="$(arg controller_yaml)" />
+        <xacro:kuroko_command_interface_position controller_yaml="$(arg controller_yaml)" />
       </xacro:if>
       <xacro:if value="${gazebo_hardware_interface=='effort'}">
-        <xacro:kuroko_transmission_effort controller_yaml="$(arg controller_yaml)" />
+        <xacro:kuroko_command_interface_effort controller_yaml="$(arg controller_yaml)" />
       </xacro:if>
     </xacro:if>
