Commit message: WIP

File: kuroko_description/xacro/gazebo/gazebo_ros2_command_interface.xacro (robot description, xacro)
@@ -12,10 +12,10 @@
       <xacro:set_position_command_interfaces joints="${['joint1','joint2']}"/>
     Full Gazebo Classic ros2_control block:
-      <xacro:gazebo_classic_ros2_control_system
+      <xacro:gazebo_ros2_control_system
           joints="${['joint1','joint2']}"
           command_if="position"
           state_ifs="${['position','velocity','effort']}"/>
-      <xacro:gazebo_classic_ros2_control_plugin
-          parameters_file="$(find your_pkg)/config/controllers.yaml"/>
+      <xacro:gazebo_ros2_control_plugin
+          controller_yaml="$(find your_pkg)/config/controllers.yaml"/>
   -->
   <!-- Internal: emit <state_interface> tags from a list -->
@@ -73,5 +73,5 @@
   </xacro:macro>
   <!-- Gazebo Classic ros2_control system (fixed to gazebo_ros2_control) -->
-  <xacro:macro name="gazebo_classic_ros2_control_system"
+  <xacro:macro name="gazebo_ros2_control_system"
                params="joints
                        command_if:='position'

Commit message: wip

File: kuroko_description/xacro/gazebo/gazebo_ros2_command_interface.xacro (robot description, xacro)
@@ -93,12 +93,8 @@
   </xacro:macro>
   <!-- Gazebo Classic plugin block (gazebo_ros2_control) -->
-  <xacro:macro name="gazebo_ros2_control_plugin" params="controller_yaml:=''">
+  <xacro:macro name="gazebo_ros2_control_plugin" params="controller_yaml">
     <gazebo>
       <plugin name="gazebo_ros2_control" filename="libgazebo_ros2_control.so">
-        <robot_param>robot_description</robot_param>
-        <robot_param_node>robot_state_publisher</robot_param_node>
-        <xacro:if value="${controller_yaml != ''}">
-          <parameters>${controller_yaml}</parameters>
-        </xacro:if>
+        <parameters>${controller_yaml}</parameters>
       </plugin>
     </gazebo>

Commit message: WIP

File: kuroko_description/xacro/gazebo/gazebo_ros2_command_interface.xacro (robot description, xacro)
@@ -1,23 +1,12 @@
-<?xml version="1.0" encoding="UTF-8"?>
+<?xml version="1.0"?>
 <robot xmlns:xacro="http://www.ros.org/wiki/xacro">
   <!--
-    Command interface generators for Gazebo Classic (gazebo_ros2_control)
-    Single joint:
-      <xacro:set_effort_command_interface joint_name="joint1"/>
-      <xacro:set_velocity_command_interface joint_name="joint1"/>
-      <xacro:set_position_command_interface joint_name="joint1"/>
-    Multiple joints:
-      <xacro:set_effort_command_interfaces joints="${['joint1','joint2']}"/>
-      <xacro:set_velocity_command_interfaces joints="${['joint1','joint2']}"/>
-      <xacro:set_position_command_interfaces joints="${['joint1','joint2']}"/>
-    Full Gazebo Classic ros2_control block:
-      <xacro:gazebo_ros2_control_system
-          joints="${['joint1','joint2']}"
-          command_if="position"
-          state_ifs="${['position','velocity','effort']}"/>
-      <xacro:gazebo_ros2_control_plugin
-          controller_yaml="$(find your_pkg)/config/controllers.yaml"/>
+    Gazebo Classic ros2_control command interfaces (no PID).
+    Provides:
+      - set_effort_command_interfaces(joints, state_ifs)
+      - set_velocity_command_interfaces(joints, state_ifs)
+      - set_position_command_interfaces(joints, state_ifs)
+      - gazebo_ros2_control_system(joints, command_if, state_ifs)
   -->
-  <!-- Internal: emit <state_interface> tags from a list -->
   <xacro:macro name="_state_interfaces_loop" params="ifs">
     <xacro:if value="${len(ifs) > 0}">
@@ -26,6 +15,6 @@
     </xacro:if>
   </xacro:macro>
-  <!-- Generic ros2_control joint block -->
-  <xacro:macro name="ros2_control_joint" params="joint_name command_if state_ifs:=${['position','velocity','effort']}">
+  <xacro:macro name="_ros2_control_joint"
+               params="joint_name command_if state_ifs:=${['position','velocity','effort']}">
     <joint name="${joint_name}">
       <command_interface name="${command_if}"/>
@@ -33,44 +22,25 @@
     </joint>
   </xacro:macro>
-  <!-- Internal: per-joint wrappers -->
-  <xacro:macro name="_effort_command_joint" params="joint_name state_ifs:=${['position','velocity','effort']}">
-    <xacro:ros2_control_joint joint_name="${joint_name}" command_if="effort" state_ifs="${state_ifs}"/>
-  </xacro:macro>
-  <xacro:macro name="_velocity_command_joint" params="joint_name state_ifs:=${['position','velocity','effort']}">
-    <xacro:ros2_control_joint joint_name="${joint_name}" command_if="velocity" state_ifs="${state_ifs}"/>
-  </xacro:macro>
-  <xacro:macro name="_position_command_joint" params="joint_name state_ifs:=${['position','velocity','effort']}">
-    <xacro:ros2_control_joint joint_name="${joint_name}" command_if="position" state_ifs="${state_ifs}"/>
-  </xacro:macro>
-  <!-- Public: single joint -->
-  <xacro:macro name="set_effort_command_interface" params="joint_name state_ifs:=${['position','velocity','effort']}">
-    <xacro:_effort_command_joint joint_name="${joint_name}" state_ifs="${state_ifs}"/>
-  </xacro:macro>
-  <xacro:macro name="set_velocity_command_interface" params="joint_name state_ifs:=${['position','velocity','effort']}">
-    <xacro:_velocity_command_joint joint_name="${joint_name}" state_ifs="${state_ifs}"/>
-  </xacro:macro>
-  <xacro:macro name="set_position_command_interface" params="joint_name state_ifs:=${['position','velocity','effort']}">
-    <xacro:_position_command_joint joint_name="${joint_name}" state_ifs="${state_ifs}"/>
-  </xacro:macro>
-  <!-- Public: multiple joints -->
-  <xacro:macro name="set_effort_command_interfaces" params="joints state_ifs:=${['position','velocity','effort']}">
+  <xacro:macro name="set_effort_command_interfaces"
+               params="joints state_ifs:=${['position','velocity','effort']}">
     <xacro:if value="${len(joints) > 0}">
-      <xacro:_effort_command_joint joint_name="${joints[0]}" state_ifs="${state_ifs}"/>
+      <xacro:_ros2_control_joint joint_name="${joints[0]}" command_if="effort" state_ifs="${state_ifs}"/>
       <xacro:set_effort_command_interfaces joints="${joints[1:]}" state_ifs="${state_ifs}"/>
     </xacro:if>
   </xacro:macro>
-  <xacro:macro name="set_velocity_command_interfaces" params="joints state_ifs:=${['position','velocity','effort']}">
+  <xacro:macro name="set_velocity_command_interfaces"
+               params="joints state_ifs:=${['position','velocity','effort']}">
     <xacro:if value="${len(joints) > 0}">
-      <xacro:_velocity_command_joint joint_name="${joints[0]}" state_ifs="${state_ifs}"/>
+      <xacro:_ros2_control_joint joint_name="${joints[0]}" command_if="velocity" state_ifs="${state_ifs}"/>
       <xacro:set_velocity_command_interfaces joints="${joints[1:]}" state_ifs="${state_ifs}"/>
     </xacro:if>
   </xacro:macro>
-  <xacro:macro name="set_position_command_interfaces" params="joints state_ifs:=${['position','velocity','effort']}">
+  <xacro:macro name="set_position_command_interfaces"
+               params="joints state_ifs:=${['position','velocity','effort']}">
     <xacro:if value="${len(joints) > 0}">
-      <xacro:_position_command_joint joint_name="${joints[0]}" state_ifs="${state_ifs}"/>
+      <xacro:_ros2_control_joint joint_name="${joints[0]}" command_if="position" state_ifs="${state_ifs}"/>
       <xacro:set_position_command_interfaces joints="${joints[1:]}" state_ifs="${state_ifs}"/>
     </xacro:if>
   </xacro:macro>
-  <!-- Gazebo Classic ros2_control system (fixed to gazebo_ros2_control) -->
   <xacro:macro name="gazebo_ros2_control_system"
                params="joints
@@ -92,11 +62,3 @@
     </ros2_control>
   </xacro:macro>
-  <!-- Gazebo Classic plugin block (gazebo_ros2_control) -->
-  <xacro:macro name="gazebo_ros2_control_plugin" params="controller_yaml">
-    <gazebo>
-      <plugin name="gazebo_ros2_control" filename="libgazebo_ros2_control.so">
-        <parameters>${controller_yaml}</parameters>
-      </plugin>
-    </gazebo>
-  </xacro:macro>
 </robot>

Commit message: Refactoring

File: kuroko_description/xacro/gazebo/gazebo_ros2_command_interface.xacro (robot description, xacro)
@@ -93,8 +93,13 @@
   </xacro:macro>
   <!-- Gazebo Classic plugin block (gazebo_ros2_control) -->
-  <xacro:macro name="gazebo_ros2_control_plugin" params="controller_yaml">
+  <xacro:macro name="gazebo_ros2_control_plugin" params="controller_yaml:='' pid_yaml:=''">
     <gazebo>
       <plugin name="gazebo_ros2_control" filename="libgazebo_ros2_control.so">
-        <parameters>${controller_yaml}</parameters>
+        <xacro:if value="${controller_yaml != ''}">
+          <parameters>${controller_yaml}</parameters>
+        </xacro:if>
+        <xacro:if value="${pid_yaml != ''}">
+          <parameters>${pid_yaml}</parameters>
+        </xacro:if>
       </plugin>
     </gazebo>

File: kuroko_description/xacro/kuroko/kuroko.xacro (robot description, xacro)
@@ -6,4 +6,5 @@
   <!-- Optional ros2_control controller parameters YAML for Gazebo Classic plugin -->
   <xacro:arg name="controller_yaml" default="$(find kuroko_description)/config/ros2_control/joint_trajectory_controller.yaml"/>
+  <xacro:arg name="pid_yaml" default="$(find kuroko_description)/config/ros2_control/gazebo_pid_gains.yaml"/>
   <xacro:property name="XACRO_DIR" value="$(find kuroko_description)/xacro" />
   <xacro:unless value="$(arg gazebo)">
@@ -67,10 +68,5 @@
     <!-- ros2_control block is always present so gazebo_ros2_control can parse robot_description.
          The Gazebo plugin itself is included only when gazebo:=true (spawned model). -->
-    <xacro:if value="${gazebo_command_interface=='position'}">
-      <xacro:kuroko_command_interface_position controller_yaml="$(arg controller_yaml)" />
-    </xacro:if>
-    <xacro:if value="${gazebo_command_interface=='effort'}">
-      <xacro:kuroko_command_interface_effort controller_yaml="$(arg controller_yaml)" />
-    </xacro:if>
+    <xacro:kuroko_command_interface_position controller_yaml="$(arg controller_yaml)" pid_yaml="$(arg pid_yaml)"/>
   </xacro:macro>
   <!-- Instantiate -->
