Commit message: Disable ROS1 gazebo plugins

File: kuroko_description/xacro/kuroko/kuroko.xacro (robot description, xacro)
@@ -3,5 +3,4 @@
   <xacro:arg name="gazebo" default="false"/>
   <xacro:arg name="box_visual" default="false"/>
-  <xacro:arg name="gazebo_motor_model" default="dc"/>
   <xacro:arg name="gazebo_hw_interface" default="position"/>
   <xacro:property name="XACRO_DIR" value="$(find kuroko_description)/xacro" />
@@ -22,25 +21,5 @@
   <xacro:include filename="${XACRO_DIR}/sensors/imu/imu_n100mini.xacro"/>
   <xacro:include filename="${XACRO_DIR}/sensors/camera/usb_camera.xacro"/>
-  <!-- MACRO:Loading Gazebo Controllers for joints -->
-  <xacro:macro name="gazebo_plugin_xacro" params="gazebo_motor_model">
-    <xacro:if value="${gazebo_motor_model=='default'}">
-      <gazebo>
-        <plugin name="gazebo_ros_control" filename="libgazebo_ros_control.so">
-          <robotNamespace>kuroko</robotNamespace>
-          <robotSimType>gazebo_ros_control/DefaultRobotHWSim</robotSimType>
-          <legacyModeNS>true</legacyModeNS>
-        </plugin>
-      </gazebo>
-    </xacro:if>
-    <xacro:if value="${gazebo_motor_model=='dc'}">
-      <gazebo>
-        <plugin name="gazebo_ros_control" filename="libgazebo_dc_motor.so">
-          <robotNamespace>kuroko</robotNamespace>
-          <robotSimType>gazebo_dc_motor/DefaultRobotHWSim</robotSimType>
-          <legacyModeNS>false</legacyModeNS>
-        </plugin>
-      </gazebo>
-    </xacro:if>
-  </xacro:macro>
+  <!-- DOTO:Loading Gazebo Controllers for joints -->
   <!-- MACRO:Setting up a Robot Model -->
   <xacro:macro name="kuroko_xacro" params="gazebo box_visual gazebo_hw_interface">
@@ -74,4 +53,3 @@
   <xacro:kuroko_xacro gazebo="$(arg gazebo)" box_visual="$(arg box_visual)"
     gazebo_hw_interface="$(arg gazebo_hw_interface)"/>
-  <xacro:gazebo_plugin_xacro gazebo_motor_model="$(arg gazebo_motor_model)"/>
 </robot>

File: kuroko_description/xacro/sensors/camera/usb_camera.xacro (robot description, xacro)
@@ -52,15 +52,5 @@
           </distortion>
         </camera>
-        <plugin name="${name}_camera_plugin" filename="libgazebo_ros_camera.so">
-          <alwaysOn>true</alwaysOn>
-          <updateRate>30</updateRate>
-          <cameraName>camera</cameraName>
-          <imageTopicName>resized/image</imageTopicName>
-          <cameraInfoTopicName>resized/camera_info</cameraInfoTopicName>
-          <frameName>${name}_optical_link</frameName>
-          <hackBaseline>0</hackBaseline>
-          <autoDistortion>true</autoDistortion>
-          <borderCrop>true</borderCrop>
-        </plugin>
+        <!-- TODO:Loading Gazebo Plugin for RGB Camera -->
       </sensor>
     </gazebo>

File: kuroko_description/xacro/sensors/depth/azure_kinect_gazebo.xacro (robot description, xacro)
@@ -26,23 +26,5 @@
           </clip>
         </camera>
-        <plugin name="depth_controller" filename="libgazebo_ros_openni_kinect.so">
-          <cameraName>${name}/depth</cameraName>
-          <alwaysOn>true</alwaysOn>
-          <updateRate>15</updateRate>
-          <imageTopicName>gazebo/rgb/image_raw</imageTopicName>
-          <cameraInfoTopicName>gazebo/rgb/camera_info</cameraInfoTopicName>
-          <depthImageTopicName>image_raw</depthImageTopicName>
-          <depthImageCameraInfoTopicName>camera_info</depthImageCameraInfoTopicName>
-          <pointCloudTopicName>gazebo/points</pointCloudTopicName>
-          <frameName>${name}_depth_optical_frame</frameName>
-          <baseline>0.1</baseline>
-          <distortion_k1>0.0</distortion_k1>
-          <distortion_k2>0.0</distortion_k2>
-          <distortion_k3>0.0</distortion_k3>
-          <distortion_t1>0.0</distortion_t1>
-          <distortion_t2>0.0</distortion_t2>
-          <pointCloudCutoff>0.25</pointCloudCutoff>
-          <pointCloudCutoffMax>3.0</pointCloudCutoffMax>
-        </plugin>
+        <!-- TODO:Loading Gazebo Plugin for Depth Camera -->
       </sensor>
     </gazebo>
@@ -64,19 +46,5 @@
           </clip>
         </camera>
-        <plugin name="rgb_controller" filename="libgazebo_ros_camera.so">
-          <cameraName>${name}/rgb_no_resized</cameraName>
-          <alwaysOn>true</alwaysOn>
-          <updateRate>0</updateRate>
-          <imageTopicName>image_raw</imageTopicName>
-          <cameraInfoTopicName>camera_info</cameraInfoTopicName>
-          <frameName>${name}_rgb_optical_frame</frameName>
-          <baseline>0.1</baseline>
-          <distortion_k1>0.0</distortion_k1>
-          <distortion_k2>0.0</distortion_k2>
-          <distortion_k3>0.0</distortion_k3>
-          <distortion_t1>0.0</distortion_t1>
-          <distortion_t2>0.0</distortion_t2>
-          <pointCloudCutoff>0.4</pointCloudCutoff>
-        </plugin>
+        <!-- TODO:Loading Gazebo Plugin for RGB Camera -->
       </sensor>
     </gazebo>

File: kuroko_description/xacro/sensors/depth/maixsense_a075v_gazebo.xacro (robot description, xacro)
@@ -23,23 +23,5 @@
           </clip>
         </camera>
-        <plugin name="depth_controller" filename="libgazebo_ros_openni_kinect.so">
-          <cameraName>${name}/depth</cameraName>
-          <alwaysOn>true</alwaysOn>
-          <updateRate>15</updateRate>
-          <imageTopicName>gazebo/rgb/image_raw</imageTopicName>
-          <cameraInfoTopicName>gazebo/rgb/camera_info</cameraInfoTopicName>
-          <depthImageTopicName>image_raw</depthImageTopicName>
-          <depthImageCameraInfoTopicName>camera_info</depthImageCameraInfoTopicName>
-          <pointCloudTopicName>gazebo/points</pointCloudTopicName>
-          <frameName>${name}_depth_optical_frame</frameName>
-          <baseline>0.1</baseline>
-          <distortion_k1>0.0</distortion_k1>
-          <distortion_k2>0.0</distortion_k2>
-          <distortion_k3>0.0</distortion_k3>
-          <distortion_t1>0.0</distortion_t1>
-          <distortion_t2>0.0</distortion_t2>
-          <pointCloudCutoff>0.2</pointCloudCutoff>
-          <pointCloudCutoffMax>2.0</pointCloudCutoffMax>
-        </plugin>
+        <!-- TODO:Loading Gazebo Plugin for Depth Camera -->
       </sensor>
     </gazebo>
@@ -61,20 +43,5 @@
           </clip>
         </camera>
-        <plugin name="rgb_controller" filename="libgazebo_ros_camera.so">
-          <cameraName>${name}/rgb_no_resized</cameraName>
-          <alwaysOn>true</alwaysOn>
-          <updateRate>0</updateRate>
-          <imageTopicName>image_raw</imageTopicName>
-          <cameraInfoTopicName>camera_info</cameraInfoTopicName>
-          <frameName>${name}_rgb_optical_frame</frameName>
-          <baseline>0.1</baseline>
-          <distortion_k1>0.0</distortion_k1>
-          <distortion_k2>0.0</distortion_k2>
-          <distortion_k3>0.0</distortion_k3>
-          <distortion_t1>0.0</distortion_t1>
-          <distortion_t2>0.0</distortion_t2>
-          <pointCloudCutoff>0.01</pointCloudCutoff>
-          <pointCloudCutoffMax>8.0</pointCloudCutoffMax>
-        </plugin>
+        <!-- TODO:Loading Gazebo Plugin for RGB Camera -->
       </sensor>
     </gazebo>

File: kuroko_description/xacro/sensors/imu/imu_n100mini_gazebo.xacro (robot description, xacro)
@@ -6,31 +6,6 @@
     </gazebo>
     <gazebo>
-      <plugin filename="libhector_gazebo_ros_imu.so" name="imu_controller">
-        <alwaysOn>true</alwaysOn>
-        <updateRate>${update_rate}</updateRate>
-        <bodyName>${name}_link</bodyName>
-        <topicName>/kuroko/sensors/imu/data</topicName>
-        <serviceName>/kuroko/sensors/imu/service</serviceName>
-        <frameId>${name}_link</frameId>
-        <gaussianNoise>0</gaussianNoise>
-        <xyzOffset>0 0 0</xyzOffset>
-        <rateOffset>0 0 0</rateOffset>
-        <rpyOffset>0 0 0</rpyOffset>
-      </plugin>
-      <plugin filename="libhector_gazebo_ros_magnetic.so" name="magnetic_controller">
-        <alwaysOn>true</alwaysOn>
-        <updateRate>${update_rate}</updateRate>
-        <bodyName>${name}_link</bodyName>
-        <topicName>/kuroko/sensors/imu/mag</topicName>
-        <frameId>${name}_link</frameId>
-        <useMagneticFieldMsgs>true</useMagneticFieldMsgs>
-        <magnitude>0.000047</magnitude>
-        <declination>-7.81</declination>
-        <inclination>49.48</inclination>
-        <offset>0 0 0</offset>
-        <drift>0 0 0</drift>
-        <driftFrequency>0 0 0</driftFrequency>
-        <gaussianNoise>0 0 0</gaussianNoise>
-      </plugin>
+      <!-- TODO:Loading Gazebo Plugin for IMU -->
+      <!-- TODO:Loading Gazebo Plugin for Magnetic Sensor -->
     </gazebo>
   </xacro:macro>

File: kuroko_description/xacro/sensors/lidar/urg.xacro (robot description, xacro)
@@ -27,8 +27,5 @@
           </noise>
         </ray>
-        <plugin name="${sensor_name}_gazebo_plugin" filename="libgazebo_ros_gpu_laser.so">
-          <frameName>${firame_id}</frameName>
-          <topicName>${topic_name}</topicName>
-        </plugin>
+        <!-- TODO:Loading Gazebo Plugin for 2D LiDAR -->
       </sensor>
     </gazebo>

File: kuroko_description/xacro/sensors/range/tfluna_gazebo.xacro (robot description, xacro)
@@ -29,13 +29,5 @@
           </range>
         </ray>
-        <plugin name="gazebo_ros_${name}_controller" filename="libgazebo_ros_range.so">
-          <gaussianNoise>0.005</gaussianNoise>
-          <alwaysOn>true</alwaysOn>
-          <updateRate>${update_rate}</updateRate>
-          <topicName>${ros_topic}</topicName>
-          <frameName>${name}_link</frameName>
-          <radiation>INFRARED</radiation>
-          <fov>${fov}</fov>
-        </plugin>
+        <!-- TODO:Loading Gazebo Plugin for Range Sensor -->
       </sensor>
     </gazebo>

Commit message: Set mesh color

File: kuroko_description/xacro/kuroko/kuroko.xacro (robot description, xacro)
@@ -6,4 +6,5 @@
   <xacro:property name="XACRO_DIR" value="$(find kuroko_description)/xacro" />
   <xacro:property name="MESH_DIR" value="package://kuroko_description/meshes" />
+  <xacro:include filename="${XACRO_DIR}/physics/materials.xacro"/>
   <xacro:include filename="${XACRO_DIR}/physics/box_physics.xacro"/>
   <xacro:include filename="${XACRO_DIR}/physics/gazebo_passive_joint.xacro"/>

File: kuroko_description/xacro/kuroko/parts/arm_l.xacro (robot description, xacro)
@@ -18,4 +18,5 @@
             <mesh filename="${MESH_DIR}/kuroko/stl/shoulder_l_pitch.stl"/>
           </geometry>
+          <material name="dark_gray"/>
         </visual>
       </xacro:unless>
@@ -41,4 +42,5 @@
             <mesh filename="${MESH_DIR}/kuroko/stl/shoulder_l_roll.stl"/>
           </geometry>
+          <material name="dark_gray"/>
         </visual>
       </xacro:unless>
@@ -64,4 +66,5 @@
             <mesh filename="${MESH_DIR}/kuroko/stl/elbow_l_front.stl"/>
           </geometry>
+          <material name="dark_gray"/>
         </visual>
       </xacro:unless>
@@ -89,4 +92,5 @@
             <mesh filename="${MESH_DIR}/kuroko/stl/elbow_l_rear.stl"/>
           </geometry>
+          <material name="dark_gray"/>
         </visual>
       </xacro:unless>

File: kuroko_description/xacro/kuroko/parts/arm_r.xacro (robot description, xacro)
@@ -18,4 +18,5 @@
             <mesh filename="${MESH_DIR}/kuroko/stl/shoulder_r_pitch.stl"/>
           </geometry>
+          <material name="dark_gray"/>
         </visual>
       </xacro:unless>
@@ -41,4 +42,5 @@
             <mesh filename="${MESH_DIR}/kuroko/stl/shoulder_r_roll.stl"/>
           </geometry>
+          <material name="dark_gray"/>
         </visual>
       </xacro:unless>
@@ -64,4 +66,5 @@
             <mesh filename="${MESH_DIR}/kuroko/stl/elbow_r_front.stl"/>
           </geometry>
+          <material name="dark_gray"/>
         </visual>
       </xacro:unless>
@@ -89,4 +92,5 @@
             <mesh filename="${MESH_DIR}/kuroko/stl/elbow_r_rear.stl"/>
           </geometry>
+          <material name="dark_gray"/>
         </visual>
       </xacro:unless>

File: kuroko_description/xacro/kuroko/parts/body.xacro (robot description, xacro)
@@ -10,4 +10,5 @@
             <mesh filename="${MESH_DIR}/kuroko/stl/waist.stl"/>
           </geometry>
+          <material name="dark_gray"/>
         </visual>
       </xacro:unless>
@@ -35,4 +36,5 @@
             <mesh filename="${MESH_DIR}/kuroko/stl/chest.stl"/>
           </geometry>
+          <material name="dark_gray"/>
         </visual>
       </xacro:unless>

File: kuroko_description/xacro/kuroko/parts/leg_l.xacro (robot description, xacro)
@@ -18,4 +18,5 @@
             <mesh filename="${MESH_DIR}/kuroko/stl/hip_l_roll.stl"/>
           </geometry>
+          <material name="dark_gray"/>
         </visual>
       </xacro:unless>
@@ -42,4 +43,5 @@
             <mesh filename="${MESH_DIR}/kuroko/stl/hip_l_pitch.stl"/>
           </geometry>
+          <material name="dark_gray"/>
         </visual>
       </xacro:unless>
@@ -66,4 +68,5 @@
             <mesh filename="${MESH_DIR}/kuroko/stl/shin_l_active.stl"/>
           </geometry>
+          <material name="dark_gray"/>
         </visual>
       </xacro:unless>
@@ -90,4 +93,5 @@
             <mesh filename="${MESH_DIR}/kuroko/stl/thigh_l_active.stl"/>
           </geometry>
+          <material name="dark_gray"/>
         </visual>
       </xacro:unless>
@@ -136,4 +140,5 @@
             <mesh filename="${MESH_DIR}/kuroko/stl/shin_r_front_passive.stl"/>
           </geometry>
+          <material name="dark_gray"/>
         </visual>
       </xacro:unless>
@@ -160,4 +165,5 @@
             <mesh filename="${MESH_DIR}/kuroko/stl/thigh_r_middle_passive.stl"/>
           </geometry>
+          <material name="dark_gray"/>
         </visual>
       </xacro:unless>
@@ -206,4 +212,5 @@
             <mesh filename="${MESH_DIR}/kuroko/stl/shin_r_rear_passive.stl"/>
           </geometry>
+          <material name="dark_gray"/>
         </visual>
       </xacro:unless>
@@ -230,4 +237,5 @@
             <mesh filename="${MESH_DIR}/kuroko/stl/knee_r_passive.stl"/>
           </geometry>
+          <material name="dark_gray"/>
         </visual>
       </xacro:unless>
@@ -280,4 +288,5 @@
             <mesh filename="${MESH_DIR}/kuroko/stl/thigh_r_rear_passive.stl"/>
           </geometry>
+          <material name="dark_gray"/>
         </visual>
       </xacro:unless>
@@ -308,4 +317,5 @@
             <mesh filename="${MESH_DIR}/kuroko/stl/ankle_r_pitch_passive.stl"/>
           </geometry>
+          <material name="dark_gray"/>
         </visual>
       </xacro:unless>
@@ -335,4 +345,5 @@
             <mesh filename="${MESH_DIR}/kuroko/stl/ankle_l_roll.stl"/>
           </geometry>
+          <material name="dark_gray"/>
         </visual>
       </xacro:unless>
@@ -359,4 +370,5 @@
             <mesh filename="${MESH_DIR}/kuroko/stl/ankle_r_yaw.stl"/>
           </geometry>
+          <material name="dark_gray"/>
         </visual>
       </xacro:unless>

File: kuroko_description/xacro/kuroko/parts/leg_r.xacro (robot description, xacro)
@@ -18,4 +18,5 @@
             <mesh filename="${MESH_DIR}/kuroko/stl/hip_r_roll.stl"/>
           </geometry>
+          <material name="dark_gray"/>
         </visual>
       </xacro:unless>
@@ -42,4 +43,5 @@
             <mesh filename="${MESH_DIR}/kuroko/stl/hip_r_pitch.stl"/>
           </geometry>
+          <material name="dark_gray"/>
         </visual>
       </xacro:unless>
@@ -66,4 +68,5 @@
             <mesh filename="${MESH_DIR}/kuroko/stl/shin_r_active.stl"/>
           </geometry>
+          <material name="dark_gray"/>
         </visual>
       </xacro:unless>
@@ -90,4 +93,5 @@
             <mesh filename="${MESH_DIR}/kuroko/stl/thigh_r_active.stl"/>
           </geometry>
+          <material name="dark_gray"/>
         </visual>
       </xacro:unless>
@@ -136,4 +140,5 @@
             <mesh filename="${MESH_DIR}/kuroko/stl/shin_r_front_passive.stl"/>
           </geometry>
+          <material name="dark_gray"/>
         </visual>
       </xacro:unless>
@@ -160,4 +165,5 @@
             <mesh filename="${MESH_DIR}/kuroko/stl/thigh_r_middle_passive.stl"/>
           </geometry>
+          <material name="dark_gray"/>
         </visual>
       </xacro:unless>
@@ -206,4 +212,5 @@
             <mesh filename="${MESH_DIR}/kuroko/stl/shin_r_rear_passive.stl"/>
           </geometry>
+          <material name="dark_gray"/>
         </visual>
       </xacro:unless>
@@ -230,4 +237,5 @@
             <mesh filename="${MESH_DIR}/kuroko/stl/knee_r_passive.stl"/>
           </geometry>
+          <material name="dark_gray"/>
         </visual>
       </xacro:unless>
@@ -280,4 +288,5 @@
             <mesh filename="${MESH_DIR}/kuroko/stl/thigh_r_rear_passive.stl"/>
           </geometry>
+          <material name="dark_gray"/>
         </visual>
       </xacro:unless>
@@ -308,4 +317,5 @@
             <mesh filename="${MESH_DIR}/kuroko/stl/ankle_r_pitch_passive.stl"/>
           </geometry>
+          <material name="dark_gray"/>
         </visual>
       </xacro:unless>
@@ -336,4 +346,5 @@
             <mesh filename="${MESH_DIR}/kuroko/stl/ankle_r_roll.stl"/>
           </geometry>
+          <material name="dark_gray"/>
         </visual>
       </xacro:unless>
@@ -360,4 +371,5 @@
             <mesh filename="${MESH_DIR}/kuroko/stl/ankle_r_yaw.stl"/>
           </geometry>
+          <material name="dark_gray"/>
         </visual>
       </xacro:unless>

Commit message: Add kuroko_gz_sim

File: kuroko_description/xacro/kuroko/kuroko.xacro (robot description, xacro)
@@ -9,6 +9,8 @@
   <xacro:include filename="${XACRO_DIR}/physics/box_physics.xacro"/>
   <xacro:include filename="${XACRO_DIR}/physics/gazebo_passive_joint.xacro"/>
+  <xacro:include filename="${XACRO_DIR}/physics/gz_sim_servo.xacro"/>
   <xacro:include filename="${XACRO_DIR}/kuroko/parts/body.xacro"/>
   <xacro:include filename="${XACRO_DIR}/kuroko/transmission/body.gazebo"/>
+  <xacro:include filename="${XACRO_DIR}/kuroko/ros2_control/body_gz_sim.xacro"/>
   <xacro:include filename="${XACRO_DIR}/kuroko/parts/arm_r.xacro"/>
   <xacro:include filename="${XACRO_DIR}/kuroko/transmission/arm_r.gazebo"/>
@@ -33,4 +35,5 @@
     <xacro:body_xacro box_visual="$(arg box_visual)"/>
     <xacro:body_gazebo gazebo_hw_interface="${gazebo_hw_interface}"/>
+    <xacro:body_gz_sim/>
     <xacro:arm_r_xacro box_visual="$(arg box_visual)"/>
     <xacro:arm_r_gazebo gazebo_hw_interface="${gazebo_hw_interface}"/>

File: kuroko_description/xacro/kuroko/parts/leg_l.xacro (robot description, xacro)
@@ -247,5 +247,5 @@
     </link>
     <xacro:if value="$(arg gazebo)">
-      <xacro:gazebo_poassive_joint name="knee_l_front_passive_loop" xyz="0.0335 0 0"
+      <xacro:gazebo_passive_joint name="knee_l_front_passive_loop" xyz="0.0335 0 0"
         parent="knee_l_passive_link" child="thigh_l_active_link" axis="0 1 0" lower="-1.8588" upper="0.4974"/>
     </xacro:if>
@@ -298,5 +298,5 @@
     </link>
     <xacro:if value="$(arg gazebo)">
-      <xacro:gazebo_poassive_joint name="thigh_l_rear_passive_loop" xyz="0 0 0.1" rpy="0 1.832597551 0"
+      <xacro:gazebo_passive_joint name="thigh_l_rear_passive_loop" xyz="0 0 0.1" rpy="0 1.832597551 0"
         parent="thigh_l_rear_passive_link" child="shin_l_active_link" axis="0 1 0"/>
     </xacro:if>
@@ -327,5 +327,5 @@
     </link>
     <xacro:if value="$(arg gazebo)">
-      <xacro:gazebo_poassive_joint name="ankle_l_front_passive_loop" xyz="0.0335 0 0" rpy="0 -0.785398163 0"
+      <xacro:gazebo_passive_joint name="ankle_l_front_passive_loop" xyz="0.0335 0 0" rpy="0 -0.785398163 0"
         parent="ankle_l_rear_passive_link" child="shin_l_front_passive_link" axis="0 1 0"/>
     </xacro:if>

File: kuroko_description/xacro/kuroko/parts/leg_r.xacro (robot description, xacro)
@@ -247,5 +247,5 @@
     </link>
     <xacro:if value="$(arg gazebo)">
-      <xacro:gazebo_poassive_joint name="knee_r_front_passive_loop" xyz="0.0335 0 0"
+      <xacro:gazebo_passive_joint name="knee_r_front_passive_loop" xyz="0.0335 0 0"
         parent="knee_r_passive_link" child="thigh_r_active_link" axis="0 1 0" lower="-1.8588" upper="0.4974"/>
     </xacro:if>
@@ -298,5 +298,5 @@
     </link>
     <xacro:if value="$(arg gazebo)">
-      <xacro:gazebo_poassive_joint name="thigh_r_rear_passive_loop" xyz="0 0 0.1" rpy="0 1.832597551 0"
+      <xacro:gazebo_passive_joint name="thigh_r_rear_passive_loop" xyz="0 0 0.1" rpy="0 1.832597551 0"
         parent="thigh_r_rear_passive_link" child="shin_r_active_link" axis="0 1 0"/>
     </xacro:if>
@@ -328,5 +328,5 @@
     </link>
     <xacro:if value="$(arg gazebo)">
-      <xacro:gazebo_poassive_joint name="ankle_r_front_passive_loop" xyz="0.0335 0 0" rpy="0 -0.785398163 0"
+      <xacro:gazebo_passive_joint name="ankle_r_front_passive_loop" xyz="0.0335 0 0" rpy="0 -0.785398163 0"
         parent="ankle_r_rear_passive_link" child="shin_r_front_passive_link" axis="0 1 0"/>
     </xacro:if>

File: kuroko_description/xacro/physics/gazebo_passive_joint.xacro (robot description, xacro)
@@ -1,5 +1,5 @@
 <?xml version="1.0"?>
 <robot xmlns:xacro="http://www.ros.org/wiki/xacro">
-  <xacro:macro name="gazebo_poassive_joint"
+  <xacro:macro name="gazebo_passive_joint"
     params="name:='joint' parent:='parent' child:='child' xyz:='0 0 0' rpy:='0 0 0' axis:='0 1 0' lower:=-3.1416 upper:=3.1416">
     <gazebo>
