Commit message: Remove transmissions for ROS1

File: kuroko_description/xacro/kuroko/kuroko.xacro (robot description, xacro)
@@ -11,14 +11,9 @@
   <xacro:include filename="${XACRO_DIR}/physics/gz_sim_servo.xacro"/>
   <xacro:include filename="${XACRO_DIR}/kuroko/parts/body.xacro"/>
-  <xacro:include filename="${XACRO_DIR}/kuroko/transmission/body.gazebo"/>
   <xacro:include filename="${XACRO_DIR}/kuroko/ros2_control/body_gz_sim.xacro"/>
   <xacro:include filename="${XACRO_DIR}/kuroko/parts/arm_r.xacro"/>
-  <xacro:include filename="${XACRO_DIR}/kuroko/transmission/arm_r.gazebo"/>
   <xacro:include filename="${XACRO_DIR}/kuroko/parts/arm_l.xacro"/>
-  <xacro:include filename="${XACRO_DIR}/kuroko/transmission/arm_l.gazebo"/>
   <xacro:include filename="${XACRO_DIR}/kuroko/parts/leg_r.xacro"/>
-  <xacro:include filename="${XACRO_DIR}/kuroko/transmission/leg_r.gazebo"/>
   <xacro:include filename="${XACRO_DIR}/kuroko/parts/leg_l.xacro"/>
-  <xacro:include filename="${XACRO_DIR}/kuroko/transmission/leg_l.gazebo"/>
   <xacro:include filename="${XACRO_DIR}/sensors/range/tfluna.xacro"/>
   <xacro:include filename="${XACRO_DIR}/sensors/imu/imu_n100mini.xacro"/>
@@ -34,14 +29,9 @@
     </joint>
     <xacro:body_xacro box_visual="$(arg box_visual)"/>
-    <xacro:body_gazebo gazebo_hw_interface="${gazebo_hw_interface}"/>
     <xacro:body_gz_sim/>
     <xacro:arm_r_xacro box_visual="$(arg box_visual)"/>
-    <xacro:arm_r_gazebo gazebo_hw_interface="${gazebo_hw_interface}"/>
     <xacro:arm_l_xacro box_visual="$(arg box_visual)"/>
-    <xacro:arm_l_gazebo gazebo_hw_interface="${gazebo_hw_interface}"/>
     <xacro:leg_r_xacro gazebo="$(arg gazebo)" box_visual="$(arg box_visual)"/>
-    <xacro:leg_r_gazebo gazebo_hw_interface="${gazebo_hw_interface}"/>
     <xacro:leg_l_xacro gazebo="$(arg gazebo)" box_visual="$(arg box_visual)"/>
-    <xacro:leg_l_gazebo gazebo_hw_interface="${gazebo_hw_interface}"/>
     <xacro:imu_n100mini parent="waist_link" name="imu">
       <origin xyz="-0.04 0 -0.01" rpy="0 0 0"/>

File: kuroko_description/xacro/physics/default_gazebo_params.xacro (robot description, xacro)
@@ -1,29 +1,4 @@
 <?xml version="1.0"?>
 <robot xmlns:xacro="http://www.ros.org/wiki/xacro">
-  <xacro:macro name="default_motor_transmission" params="joint_name gazebo_hw_interface">
-    <gazebo reference="${joint_name}">
-      <implicitSpringDamper>1</implicitSpringDamper>
-    </gazebo>
-    <transmission name="${joint_name}_trans">
-      <type>transmission_interface/SimpleTransmission</type>
-      <joint name="${joint_name}">
-        <xacro:if value="${gazebo_hw_interface=='effort'}">
-          <hardwareInterface>hardware_interface/EffortJointInterface</hardwareInterface>
-        </xacro:if>
-        <xacro:if value="${gazebo_hw_interface=='position'}">
-          <hardwareInterface>hardware_interface/PositionJointInterface</hardwareInterface>
-        </xacro:if>
-      </joint>
-      <actuator name="${joint_name}_motor">
-        <xacro:if value="${gazebo_hw_interface=='effort'}">
-          <hardwareInterface>hardware_interface/EffortJointInterface</hardwareInterface>
-        </xacro:if>
-        <xacro:if value="${gazebo_hw_interface=='position'}">
-          <hardwareInterface>hardware_interface/PositionJointInterface</hardwareInterface>
-        </xacro:if>
-        <mechanicalReduction>1</mechanicalReduction>
-      </actuator>
-    </transmission>
-  </xacro:macro>
   <xacro:macro name="default_link_collision" params="link_name friction">
     <gazebo reference="${link_name}">
@@ -38,20 +13,4 @@
     </gazebo>
   </xacro:macro>
-  <xacro:macro name="implicit_joint" params="joint_name">
-    <gazebo reference="${joint_name}">
-      <physics>
-        <ode>
-          <implicit_spring_damper>1</implicit_spring_damper>
-          <cfm_damping>0</cfm_damping>
-          <cfm>1e-7</cfm>
-          <erp>0.8</erp>
-          <limit>
-            <cfm>1e-7</cfm>
-            <erp>0.8</erp>
-          </limit>
-        </ode>
-      </physics>
-    </gazebo>
-  </xacro:macro>
   <xacro:macro name="preserve_fixed_joint" params="joint_name">
     <gazebo reference="${joint_name}">

Commit message: Enable IMU and Camera

File: kuroko_description/xacro/kuroko/kuroko.xacro (robot description, xacro)
@@ -20,5 +20,7 @@
   <xacro:include filename="${XACRO_DIR}/kuroko/gazebo/leg_l.gazebo"/>
   <xacro:include filename="${XACRO_DIR}/sensors/range/tfluna.xacro"/>
+  <xacro:include filename="${XACRO_DIR}/sensors/imu/enable_gz_imu_plugin.xacro"/>
   <xacro:include filename="${XACRO_DIR}/sensors/imu/imu_n100mini.xacro"/>
+  <xacro:include filename="${XACRO_DIR}/sensors/camera/enable_gz_rendering_plugin.xacro"/>
   <xacro:include filename="${XACRO_DIR}/sensors/camera/usb_camera.xacro"/>
   <!-- <xacro:include filename="${XACRO_DIR}/kuroko/ros2_control/gz_sim_trajectory_control.xacro"/> -->
@@ -43,8 +45,8 @@
     <xacro:leg_l_xacro gazebo="$(arg gazebo)" box_visual="$(arg box_visual)"/>
     <xacro:leg_l_gazebo/>
-    <xacro:imu_n100mini parent="waist_link" name="imu">
+    <xacro:imu_n100mini parent="waist_link" name="imu" namespace="/kuroko/sensors/imu">
       <origin xyz="-0.04 0 -0.01" rpy="0 0 0"/>
     </xacro:imu_n100mini>
-    <xacro:usb_camera parent="waist_link" name="camera">
+    <xacro:usb_camera parent="waist_link" name="camera" namespace="/kuroko/sensors/camera">
       <origin xyz="0.07 0 -0.026" rpy="0 0 0"/>
     </xacro:usb_camera>
@@ -54,4 +56,6 @@
     <!-- <xacro:gz_sim_trajectory_control/> -->
     <xacro:gz_sim_position_control/>
+    <xacro:enable_gz_rendering_plugin/>
+    <xacro:enable_gz_imu_plugin/>
   </xacro:macro>
   <!-- Load Macros -->

File: kuroko_description/xacro/sensors/camera/usb_camera.xacro (robot description, xacro)
@@ -1,5 +1,5 @@
 <?xml version="1.0" encoding="UTF-8"?>
 <robot xmlns:xacro="http://www.ros.org/wiki/xacro">
-  <xacro:macro name="usb_camera" params="name:='camera' parent:='base_link' *origin">
+  <xacro:macro name="usb_camera" params="name:='camera' parent:='base_link' *origin namespace">
     <xacro:property name="mount_to_camera_offset" value="0.001"/>
     <xacro:property name="size_depth" value="0.002"/>
@@ -36,5 +36,9 @@
     <!-- gazebo for camera -->
     <gazebo reference="${name}_frame_link">
-      <sensor type="camera" name="camera_camera_cam">
+      <sensor type="camera" name="${name}">
+        <always_on>true</always_on>
+        <update_rate>15.0</update_rate>
+        <topic>${namespace}/image_raw</topic>
+        <gz_frame_id>${name}_optical_link</gz_frame_id>
         <camera name="camera">
           <horizontal_fov>2.20</horizontal_fov>
@@ -42,5 +46,5 @@
             <width>384</width>
             <height>216</height>
-            <format>B8G8R8</format>
+            <format>R8G8B8</format>
           </image>
           <distortion>
@@ -52,5 +56,4 @@
           </distortion>
         </camera>
-        <!-- TODO:Loading Gazebo Plugin for RGB Camera -->
       </sensor>
     </gazebo>

File: kuroko_description/xacro/sensors/imu/imu_n100mini.xacro (robot description, xacro)
@@ -1,9 +1,6 @@
 <?xml version="1.0" encoding="UTF-8"?>
-<robot xmlns:sensor="http://playerstage.sourceforge.net/gazebo/xmlschema/#sensor"
-  xmlns:controller="http://playerstage.sourceforge.net/gazebo/xmlschema/#controller"
-  xmlns:interface="http://playerstage.sourceforge.net/gazebo/xmlschema/#interface"
-  xmlns:xacro="http://www.ros.org/wiki/xacro">
+<robot xmlns:xacro="http://www.ros.org/wiki/xacro">
   <xacro:include filename="imu_n100mini_gazebo.xacro"/>
-  <xacro:macro name="imu_n100mini" params="name parent:='base_link' update_rate:=400 *origin">
+  <xacro:macro name="imu_n100mini" params="name parent:='base_link' update_rate:=400 *origin namespace">
     <xacro:property name="depth" value="0.01"/>
     <xacro:property name="width" value="0.01"/>
@@ -37,5 +34,5 @@
       <preserveFixedJoint>true</preserveFixedJoint>
     </gazebo>
-    <xacro:n100mini_gazebo name="${name}" update_rate="${update_rate}"/>
+    <xacro:n100mini_gazebo name="${name}" update_rate="${update_rate}" namespace="${namespace}"/>
   </xacro:macro>
 </robot>

File: kuroko_description/xacro/sensors/imu/imu_n100mini_gazebo.xacro (robot description, xacro)
@@ -1,11 +1,19 @@
 <?xml version="1.0" encoding="UTF-8"?>
 <robot xmlns:xacro="http://www.ros.org/wiki/xacro">
-  <xacro:macro name="n100mini_gazebo" params="name update_rate">
+  <xacro:macro name="n100mini_gazebo" params="namespace name update_rate">
     <gazebo reference="${name}_link">
       <material>Gazebo/Gray</material>
-    </gazebo>
-    <gazebo>
-      <!-- TODO:Loading Gazebo Plugin for IMU -->
-      <!-- TODO:Loading Gazebo Plugin for Magnetic Sensor -->
+      <sensor name="imu" type="imu">
+        <always_on>true</always_on>
+        <update_rate>${update_rate}</update_rate>
+        <topic>${namespace}/data</topic>
+        <gz_frame_id>${name}_link</gz_frame_id>
+      </sensor>
+      <sensor name="magnetometer" type="magnetometer">
+        <always_on>true</always_on>
+        <update_rate>${update_rate}</update_rate>
+        <topic>${namespace}/mag</topic>
+        <gz_frame_id>${name}_link</gz_frame_id>
+      </sensor>
     </gazebo>
   </xacro:macro>

Commit message: Select controller from kuroko_gz_sim.launch.py
Fix bug

File: kuroko_description/xacro/kuroko/kuroko.xacro (robot description, xacro)
@@ -3,7 +3,8 @@
   <xacro:arg name="gazebo" default="false"/>
   <xacro:arg name="box_visual" default="false"/>
-  <xacro:arg name="gazebo_hw_interface" default="position"/>
-  <xacro:property name="XACRO_DIR" value="$(find kuroko_description)/xacro" />
-  <xacro:property name="MESH_DIR" value="package://kuroko_description/meshes" />
+  <xacro:arg name="use_pid" default="true"/>
+  <xacro:arg name="use_position_control" default="true"/>
+  <xacro:property name="XACRO_DIR" value="$(find kuroko_description)/xacro"/>
+  <xacro:property name="MESH_DIR" value="package://kuroko_description/meshes"/>
   <xacro:include filename="${XACRO_DIR}/physics/materials.xacro"/>
   <xacro:include filename="${XACRO_DIR}/physics/box_physics.xacro"/>
@@ -26,5 +27,5 @@
   <!-- DOTO:Loading Gazebo Controllers for joints -->
   <!-- MACRO:Setting up a Robot Model -->
-  <xacro:macro name="kuroko_xacro" params="gazebo box_visual gazebo_hw_interface">
+  <xacro:macro name="kuroko_xacro" params="gazebo box_visual use_pid use_position_control">
     <link name="body_link"/>
     <joint name="root_joint" type="fixed">
@@ -43,4 +44,5 @@
     <xacro:leg_l_xacro gazebo="$(arg gazebo)" box_visual="$(arg box_visual)"/>
     <xacro:leg_l_gazebo/>
+    <!-- Sensors -->
     <xacro:imu_n100mini parent="waist_link" name="imu" namespace="/kuroko/sensors/imu">
       <origin xyz="-0.04 0 -0.01" rpy="0 0 0"/>
@@ -52,6 +54,4 @@
       <origin xyz="0.07 0 -0.044" rpy="0 0 0"/>
     </xacro:tfluna>
-    <!-- <xacro:gz_sim_trajectory_control/> -->
-    <xacro:gz_sim_position_control/>
     <xacro:enable_gz_rendering_plugin/>
     <xacro:enable_gz_imu_plugin/>
@@ -80,4 +80,4 @@
   <!-- Load Macros -->
   <xacro:kuroko_xacro gazebo="$(arg gazebo)" box_visual="$(arg box_visual)"
-    gazebo_hw_interface="$(arg gazebo_hw_interface)"/>
+    use_pid="$(arg use_pid)" use_position_control="$(arg use_position_control)"/>
 </robot>
