Commit message: WIP

File: kuroko_description/xacro/kuroko/kuroko.xacro (robot description, xacro)
@@ -41,7 +41,7 @@
     <xacro:arm_l_gazebo/>
     <xacro:leg_r_xacro gazebo="$(arg gazebo)" box_visual="$(arg box_visual)"/>
-    <!-- <xacro:leg_r_gazebo/> -->
-    <!-- <xacro:leg_l_xacro gazebo="$(arg gazebo)" box_visual="$(arg box_visual)"/> -->
-    <!-- <xacro:leg_l_gazebo/> -->
+    <xacro:leg_r_gazebo/>
+    <xacro:leg_l_xacro gazebo="$(arg gazebo)" box_visual="$(arg box_visual)"/>
+    <xacro:leg_l_gazebo/>
     <!-- Sensors -->
     <xacro:imu_n100mini parent="waist_link" name="imu" namespace="/kuroko/sensors/imu">

File: kuroko_description/xacro/kuroko/parts/leg_l.xacro (robot description, xacro)
@@ -1,5 +1,5 @@
 <?xml version="1.0"?>
 <robot xmlns:xacro="http://www.ros.org/wiki/xacro">
-  <xacro:macro name="leg_l_xacro" params="gazebo:=false box_visual:=false robot_name:=kuroko">
+  <xacro:macro name="leg_l_xacro" params="gazebo:=false box_visual:=false">
     <!-- Link conencts from body. Hip first. -->
     <joint name="hip_l_roll" type="revolute">
@@ -78,67 +78,28 @@
         mass="0.008"/>
     </link>
-    <xacro:unless value="$(arg gazebo)">
-      <joint name="thigh_l_active" type="revolute">
-        <parent link="hip_l_pitch_link"/>
-        <child link="thigh_l_active_link"/>
-        <origin xyz="0.015 0.02925 -0.0305" rpy="0 -0.785398163 0"/>
-        <axis xyz="0 1 0"/>
-        <limit effort="8.9" lower="-0.4974" upper="1.8588" velocity="6.9"/>
-        <dynamics damping="1.29" friction="0.0"/>
-      </joint>
-      <link name="thigh_l_active_link">
-        <xacro:unless value="$(arg box_visual)">
-          <visual>
-            <origin xyz="0 0 0" rpy="0 0 0"/>
-            <geometry>
-              <mesh filename="${MESH_DIR}/kuroko/stl/thigh_l_active.stl"/>
-            </geometry>
-            <material name="dark_gray"/>
-          </visual>
-        </xacro:unless>
-        <xacro:if value="$(arg box_visual)">
-          <xacro:box_visual xyz="0 0 -0.05" rpy="0 0 0" size="0.014 0.0445 0.114"/>
-        </xacro:if>
-        <xacro:box_collision xyz="0 0 -0.05" rpy="0 0 0" size="0.014 0.0445 0.114"/>
-        <xacro:box_inertial xyz="0 0 -0.05" rpy="0 0 0" size="0.014 0.0445 0.114" mass="0.012"/>
-      </link>
-    </xacro:unless>
-    <!-- Split link and connect with DetachableJoint -->
-    <xacro:if value="$(arg gazebo)">
-      <joint name="thigh_l_active" type="revolute">
-        <parent link="hip_l_pitch_link"/>
-        <child link="thigh_l_active_upper_link"/>
-        <origin xyz="0.015 0.02925 -0.0305" rpy="0 -0.785398163 0"/>
-        <axis xyz="0 1 0"/>
-        <limit effort="8.9" lower="-0.4974" upper="1.8588" velocity="6.9"/>
-        <dynamics damping="1.29" friction="0.0"/>
-      </joint>
-      <link name="thigh_l_active_link">
-        <xacro:unless value="$(arg box_visual)">
-          <visual>
-            <origin xyz="0 0 0" rpy="0 0 0"/>
-            <geometry>
-              <mesh filename="${MESH_DIR}/kuroko/stl/thigh_l_active.stl"/>
-            </geometry>
-            <material name="dark_gray"/>
-          </visual>
-        </xacro:unless>
-        <xacro:if value="$(arg box_visual)">
-          <xacro:box_visual xyz="0 0 -0.05" rpy="0 0 0" size="0.014 0.0445 0.114"/>
-        </xacro:if>
-        <xacro:box_collision xyz="0 0 -0.05" rpy="0 0 0" size="0.014 0.0445 0.114"/>
-        <xacro:box_inertial xyz="0 0 -0.05" rpy="0 0 0" size="0.014 0.0445 0.114" mass="0.012"/>
-      </link>
-      <link name="thigh_l_active_lower_link">
-        <xacro:box_inertial xyz="0 0 -0.05" rpy="0 0 0" size="0.014 0.0445 0.114" mass="0.006"/>
-      </link>
-      <gazebo>
-        <plugin filename="libgz-sim-detachable-joint-system.so" name="gz::sim::systems::DetachableJoint">
-          <parent_link>thigh_l_active_upper_link</parent_link>
-          <child_model>${robot_name}</child_model>
-          <child_link>thigh_l_active_lower_link</child_link>
-        </plugin>
-      </gazebo>
-    </xacro:if>
+    <joint name="thigh_l_active" type="revolute">
+      <parent link="hip_l_pitch_link"/>
+      <child link="thigh_l_active_link"/>
+      <origin xyz="0.015 0.02925 -0.0305" rpy="0 -0.785398163 0"/>
+      <axis xyz="0 1 0"/>
+      <limit effort="8.9" lower="-0.4974" upper="1.8588" velocity="6.9"/>
+      <dynamics damping="1.29" friction="0.0"/>
+    </joint>
+    <link name="thigh_l_active_link">
+      <xacro:unless value="$(arg box_visual)">
+        <visual>
+          <origin xyz="0 0 0" rpy="0 0 0"/>
+          <geometry>
+            <mesh filename="${MESH_DIR}/kuroko/stl/thigh_l_active.stl"/>
+          </geometry>
+          <material name="dark_gray"/>
+        </visual>
+      </xacro:unless>
+      <xacro:if value="$(arg box_visual)">
+        <xacro:box_visual xyz="0 0 -0.05" rpy="0 0 0" size="0.014 0.0445 0.114"/>
+      </xacro:if>
+      <xacro:box_collision xyz="0 0 -0.05" rpy="0 0 0" size="0.014 0.0445 0.114"/>
+      <xacro:box_inertial xyz="0 0 -0.05" rpy="0 0 0" size="0.014 0.0445 0.114" mass="0.012"/>
+    </link>
     <xacro:unless value="$(arg gazebo)">
       <joint name="shin_l_front_mimic" type="revolute">
@@ -164,6 +125,6 @@
     <xacro:if value="$(arg gazebo)">
       <joint name="shin_l_front_passive" type="revolute">
-        <parent link="thigh_l_active_lower_link"/>
-        <child link="shin_l_front_passive_upper_link"/>
+        <parent link="thigh_l_active_link"/>
+        <child link="shin_l_front_passive_link"/>
         <origin xyz="0 0 -0.1" rpy="0 1.570796327 0"/>
         <axis xyz="0 1 0"/>
@@ -172,50 +133,20 @@
       </joint>
     </xacro:if>
-    <xacro:unless value="$(arg gazebo)">
-      <link name="shin_l_front_passive_link">
-        <xacro:unless value="$(arg box_visual)">
-          <visual>
-            <origin xyz="0 0 0" rpy="0 0 0"/>
-            <geometry>
-              <mesh filename="${MESH_DIR}/kuroko/stl/shin_r_front_passive.stl"/>
-            </geometry>
-            <material name="dark_gray"/>
-          </visual>
-        </xacro:unless>
-        <xacro:if value="$(arg box_visual)">
-          <xacro:box_visual xyz="0 0 -0.05" rpy="0 0 0" size="0.014 0.0385 0.114"/>
-        </xacro:if>
-        <xacro:box_collision xyz="0 0 -0.05" rpy="0 0 0" size="0.014 0.0385 0.114"/>
-        <xacro:box_inertial xyz="0 0 -0.05" rpy="0 0 0" size="0.014 0.0385 0.114" mass="0.013"/>
-      </link>
-    </xacro:unless>
-    <xacro:if value="$(arg gazebo)">
-      <link name="shin_l_front_passive_upper_link">
-        <xacro:unless value="$(arg box_visual)">
-          <visual>
-            <origin xyz="0 0 0" rpy="0 0 0"/>
-            <geometry>
-              <mesh filename="${MESH_DIR}/kuroko/stl/shin_r_front_passive.stl"/>
-            </geometry>
-            <material name="dark_gray"/>
-          </visual>
-        </xacro:unless>
-        <xacro:if value="$(arg box_visual)">
-          <xacro:box_visual xyz="0 0 -0.05" rpy="0 0 0" size="0.014 0.0385 0.114"/>
-        </xacro:if>
-        <xacro:box_collision xyz="0 0 -0.05" rpy="0 0 0" size="0.014 0.0385 0.114"/>
-        <xacro:box_inertial xyz="0 0 -0.05" rpy="0 0 0" size="0.014 0.0385 0.114" mass="0.013"/>
-      </link>
-      <link name="shin_l_front_passive_lower_link">
-        <xacro:box_inertial xyz="0 0 -0.05" rpy="0 0 0" size="0.014 0.0385 0.114" mass="0.013"/>
-      </link>
-      <gazebo>
-        <plugin filename="libgz-sim-detachable-joint-system.so" name="gz::sim::systems::DetachableJoint">
-          <parent_link>shin_l_front_passive_upper_link</parent_link>
-          <child_model>${robot_name}</child_model>
-          <child_link>shin_l_front_passive_lower_link</child_link>
-        </plugin>
-      </gazebo>
-    </xacro:if>
+    <link name="shin_l_front_passive_link">
+      <xacro:unless value="$(arg box_visual)">
+        <visual>
+          <origin xyz="0 0 0" rpy="0 0 0"/>
+          <geometry>
+            <mesh filename="${MESH_DIR}/kuroko/stl/shin_r_front_passive.stl"/>
+          </geometry>
+          <material name="dark_gray"/>
+        </visual>
+      </xacro:unless>
+      <xacro:if value="$(arg box_visual)">
+        <xacro:box_visual xyz="0 0 -0.05" rpy="0 0 0" size="0.014 0.0385 0.114"/>
+      </xacro:if>
+      <xacro:box_collision xyz="0 0 -0.05" rpy="0 0 0" size="0.014 0.0385 0.114"/>
+      <xacro:box_inertial xyz="0 0 -0.05" rpy="0 0 0" size="0.014 0.0385 0.114" mass="0.013"/>
+    </link>
     <joint name="thigh_l_middle_passive" type="revolute">
       <parent link="hip_l_pitch_link"/>
@@ -317,5 +248,5 @@
     <xacro:if value="$(arg gazebo)">
       <xacro:gazebo_passive_joint name="knee_l_front_passive_loop" xyz="0.0335 0 0"
-        parent="knee_l_passive_link" child="thigh_l_active_lower_link" axis="0 1 0" lower="-1.8588" upper="0.4974"/>
+        parent="knee_l_passive_link" child="thigh_l_active_link" axis="0 1 0" lower="-1.8588" upper="0.4974"/>
     </xacro:if>
     <xacro:unless value="$(arg gazebo)">
@@ -343,5 +274,5 @@
       <joint name="thigh_l_rear_passive" type="revolute">
         <parent link="shin_l_rear_passive_link"/>
-        <child link="thigh_l_rear_passive_upper_link"/>
+        <child link="thigh_l_rear_passive_link"/>
         <origin xyz="-0.00776457 0 -0.0289778" rpy="0 -1.570796327 0"/>
         <axis xyz="0 1 0"/>
@@ -350,53 +281,23 @@
       </joint>
     </xacro:if>
-    <xacro:unless value="$(arg gazebo)">
-      <link name="thigh_l_rear_passive_link">
-        <xacro:unless value="$(arg box_visual)">
-          <visual>
-            <origin xyz="0 0 0.1" rpy="0 0 0"/>
-            <geometry>
-              <mesh filename="${MESH_DIR}/kuroko/stl/thigh_r_rear_passive.stl"/>
-            </geometry>
-            <material name="dark_gray"/>
-          </visual>
-        </xacro:unless>
-        <xacro:if value="$(arg box_visual)">
-          <xacro:box_visual xyz="0 0 0.05" rpy="0 0 0" size="0.014 0.0285 0.114"/>
-        </xacro:if>
-        <xacro:box_collision xyz="0 0 0.05" rpy="0 0 0" size="0.014 0.0285 0.114"/>
-        <xacro:box_inertial xyz="0 0 0.05" rpy="0 0 0" size="0.014 0.0285 0.114" mass="0.011"/>
-      </link>
-    </xacro:unless>
-    <xacro:if value="$(arg gazebo)">
-      <link name="thigh_l_rear_passive_upper_link">
-        <xacro:unless value="$(arg box_visual)">
-          <visual>
-            <origin xyz="0 0 0.1" rpy="0 0 0"/>
-            <geometry>
-              <mesh filename="${MESH_DIR}/kuroko/stl/thigh_r_rear_passive.stl"/>
-            </geometry>
-            <material name="dark_gray"/>
-          </visual>
-        </xacro:unless>
-        <xacro:if value="$(arg box_visual)">
-          <xacro:box_visual xyz="0 0 0.05" rpy="0 0 0" size="0.014 0.0285 0.114"/>
-        </xacro:if>
-        <xacro:box_collision xyz="0 0 0.05" rpy="0 0 0" size="0.014 0.0285 0.114"/>
-        <xacro:box_inertial xyz="0 0 0.05" rpy="0 0 0" size="0.014 0.0285 0.114" mass="0.011"/>
-      </link>
-      <link name="thigh_l_rear_passive_lower_link">
-        <xacro:box_inertial xyz="0 0 0.05" rpy="0 0 0" size="0.014 0.0285 0.114" mass="0.011"/>
-      </link>
-      <gazebo>
-        <plugin filename="libgz-sim-detachable-joint-system.so" name="gz::sim::systems::DetachableJoint">
-          <parent_link>thigh_l_rear_passive_upper_link</parent_link>
-          <child_model>${robot_name}</child_model>
-          <child_link>thigh_l_rear_passive_lower_link</child_link>
-        </plugin>
-      </gazebo>
-    </xacro:if>
+    <link name="thigh_l_rear_passive_link">
+      <xacro:unless value="$(arg box_visual)">
+        <visual>
+          <origin xyz="0 0 0.1" rpy="0 0 0"/>
+          <geometry>
+            <mesh filename="${MESH_DIR}/kuroko/stl/thigh_r_rear_passive.stl"/>
+          </geometry>
+          <material name="dark_gray"/>
+        </visual>
+      </xacro:unless>
+      <xacro:if value="$(arg box_visual)">
+        <xacro:box_visual xyz="0 0 0.05" rpy="0 0 0" size="0.014 0.0285 0.114"/>
+      </xacro:if>
+      <xacro:box_collision xyz="0 0 0.05" rpy="0 0 0" size="0.014 0.0285 0.114"/>
+      <xacro:box_inertial xyz="0 0 0.05" rpy="0 0 0" size="0.014 0.0285 0.114" mass="0.011"/>
+    </link>
     <xacro:if value="$(arg gazebo)">
       <xacro:gazebo_passive_joint name="thigh_l_rear_passive_loop" xyz="0 0 0.1" rpy="0 1.832597551 0"
-        parent="thigh_l_rear_passive_upper_link" child="shin_l_active_link" axis="0 1 0"/>
+        parent="thigh_l_rear_passive_link" child="shin_l_active_link" axis="0 1 0"/>
     </xacro:if>
     <joint name="ankle_l_rear_passive" type="revolute">
@@ -427,5 +328,5 @@
     <xacro:if value="$(arg gazebo)">
       <xacro:gazebo_passive_joint name="ankle_l_front_passive_loop" xyz="0.0335 0 0" rpy="0 -0.785398163 0"
-        parent="ankle_l_rear_passive_link" child="shin_l_front_passive_lower_link" axis="0 1 0"/>
+        parent="ankle_l_rear_passive_link" child="shin_l_front_passive_link" axis="0 1 0"/>
     </xacro:if>
     <joint name="ankle_l_roll" type="revolute">
