Commit message: WIP

File: kuroko_description/xacro/kuroko/parts/leg_r.xacro (robot description, xacro)
@@ -78,56 +78,28 @@
       <xacro:box_inertial xyz="0 0 -0.05" rpy="0 0 0" size="0.014 0.0345 0.114" mass="0.012"/>
     </link>
-    <xacro:unless value="${split_chain}">
-      <joint name="thigh_r_active" type="revolute">
-        <parent link="hip_r_pitch_link"/>
-        <child link="thigh_r_active_link"/>
-        <origin xyz="0.015 -0.02925 -0.0305" rpy="0 -0.785398163 0"/>
-        <axis xyz="0 1 0"/>
-        <limit effort="8.9" lower="-0.4974" upper="1.8588" velocity="6.9"/>
-        <dynamics damping="1.29" friction="0.0"/>
-      </joint>
-      <link name="thigh_r_active_link">
-        <xacro:unless value="${box_visual}">
-          <visual>
-            <origin xyz="0 0 0" rpy="0 0 0"/>
-            <geometry>
-              <mesh filename="${MESH_DIR}/kuroko/stl/thigh_r_active.stl"/>
-            </geometry>
-            <material name="dark_gray"/>
-          </visual>
-        </xacro:unless>
-        <xacro:if value="${box_visual}">
-          <xacro:box_visual xyz="0 0 -0.05" rpy="0 0 0" size="0.014 0.0445 0.114"/>
-        </xacro:if>
-        <xacro:box_collision xyz="0 0 -0.05" rpy="0 0 0" size="0.014 0.0445 0.114"/>
-        <xacro:box_inertial xyz="0 0 -0.05" rpy="0 0 0" size="0.014 0.0445 0.114" mass="0.012"/>
-      </link>
-    </xacro:unless>
-    <xacro:if value="${split_chain}">
-      <joint name="thigh_r_active" type="revolute">
-        <parent link="hip_r_pitch_link"/>
-        <child link="thigh_r_active_upper_link"/>
-        <origin xyz="0.015 -0.02925 -0.0305" rpy="0 -0.785398163 0"/>
-        <axis xyz="0 1 0"/>
-        <limit effort="8.9" lower="-0.4974" upper="1.8588" velocity="6.9"/>
-        <dynamics damping="1.29" friction="0.0"/>
-      </joint>
-      <link name="thigh_r_active_upper_link">
-        <xacro:unless value="${box_visual}">
-          <visual>
-            <origin xyz="0 0 0" rpy="0 0 0"/>
-            <geometry>
-              <mesh filename="${MESH_DIR}/kuroko/stl/thigh_r_active.stl"/>
-            </geometry>
-            <material name="dark_gray"/>
-          </visual>
-        </xacro:unless>
-        <xacro:if value="${box_visual}">
-          <xacro:box_visual xyz="0 0 -0.05" rpy="0 0 0" size="0.014 0.0445 0.114"/>
-        </xacro:if>
-        <xacro:box_collision xyz="0 0 -0.05" rpy="0 0 0" size="0.014 0.0445 0.114"/>
-        <xacro:box_inertial xyz="0 0 -0.05" rpy="0 0 0" size="0.014 0.0445 0.114" mass="0.006"/>
-      </link>
-    </xacro:if>
+    <joint name="thigh_r_active" type="revolute">
+      <parent link="hip_r_pitch_link"/>
+      <child link="thigh_r_active_upper_link"/>
+      <origin xyz="0.015 -0.02925 -0.0305" rpy="0 -0.785398163 0"/>
+      <axis xyz="0 1 0"/>
+      <limit effort="8.9" lower="-0.4974" upper="1.8588" velocity="6.9"/>
+      <dynamics damping="1.29" friction="0.0"/>
+    </joint>
+    <link name="thigh_r_active_upper_link">
+      <xacro:unless value="${box_visual}">
+        <visual>
+          <origin xyz="0 0 0" rpy="0 0 0"/>
+          <geometry>
+            <mesh filename="${MESH_DIR}/kuroko/stl/thigh_r_active.stl"/>
+          </geometry>
+          <material name="dark_gray"/>
+        </visual>
+      </xacro:unless>
+      <xacro:if value="${box_visual}">
+        <xacro:box_visual xyz="0 0 -0.05" rpy="0 0 0" size="0.014 0.0445 0.114"/>
+      </xacro:if>
+      <xacro:box_collision xyz="0 0 -0.05" rpy="0 0 0" size="0.014 0.0445 0.114"/>
+      <xacro:box_inertial xyz="0 0 -0.05" rpy="0 0 0" size="0.014 0.0445 0.114" mass="0.006"/>
+    </link>
     <joint name="knee_r_rear_passive" type="revolute">
       <parent link="thigh_r_middle_passive_link"/>
@@ -173,20 +145,240 @@
       </plugin>
     </gazebo>
-    <!-- <xacro:if value="${gazebo}">
-      <xacro:unless value="${split_chain}">
-        <xacro:gazebo_passive_joint name="knee_r_front_passive_loop" xyz="0.0335 0 0"
-          parent="knee_r_passive_link" child="thigh_r_active_lower_link" axis="0 1 0" lower="-1.8588" upper="0.4974"/>
-      </xacro:unless>
-      <xacro:if value="${split_chain}">
-        <joint name="knee_r_front_passive_loop" type="revolute">
-          <parent link="knee_r_passive_link"/>
-          <child link="thigh_r_active_lower_link"/>
-          <origin xyz="0.0335 0 0" rpy="0 -0.785398164 0"/>
-          <axis xyz="0 1 0"/>
-          <limit effort="0" lower="-0.4974" upper="1.8588" velocity="1000.0"/>
-          <dynamics damping="0.0" friction="0.0"/>
-        </joint>
-      </xacro:if>
-    </xacro:if> -->
+    <joint name="shin_r_active" type="revolute">
+      <parent link="hip_r_pitch_link"/>
+      <child link="shin_r_active_link"/>
+      <origin xyz="-0.0185 -0.02925 -0.0305" rpy="0 1.047197551 0"/>
+      <axis xyz="0 1 0"/>
+      <limit effort="8.9" lower="-1.8588" upper="0.4974" velocity="6.9"/>
+      <dynamics damping="1.29" friction="0.0"/>
+    </joint>
+    <link name="shin_r_active_link">
+      <xacro:unless value="$(arg box_visual)">
+        <visual>
+          <origin xyz="0 0 0" rpy="0 0 0"/>
+          <geometry>
+            <mesh filename="${MESH_DIR}/kuroko/stl/shin_r_active.stl"/>
+          </geometry>
+          <material name="dark_gray"/>
+        </visual>
+      </xacro:unless>
+      <xacro:if value="$(arg box_visual)">
+        <xacro:box_visual xyz="-0.004745 0 -0.015" rpy="0 0 0" size="0.02349 0.0445 0.044"/>
+      </xacro:if>
+      <xacro:box_collision xyz="-0.004745 0 -0.015" rpy="0 0 0" size="0.02349 0.0445 0.044"/>
+      <xacro:box_inertial xyz="-0.004745 0 -0.015" rpy="0 0 0" size="0.02349 0.0445 0.044"
+        mass="0.008"/>
+    </link>
+    <joint name="thigh_r_rear_passive" type="revolute">
+      <parent link="shin_r_active_link"/>
+      <child link="thigh_r_rear_passive_upper_link"/>
+      <origin xyz="0 0 -0.03" rpy="0 -1.832595714 0"/>
+      <axis xyz="0 1 0"/>
+      <limit effort="0" lower="-0.9948" upper="1.832595714" velocity="1000.0"/>
+      <dynamics damping="0.0" friction="0.0"/>
+    </joint>
+    <link name="thigh_r_rear_passive_upper_link">
+      <xacro:unless value="$(arg box_visual)">
+        <visual>
+          <origin xyz="0 0 0" rpy="0 0 0"/>
+          <geometry>
+            <mesh filename="${MESH_DIR}/kuroko/stl/thigh_r_rear_passive.stl"/>
+          </geometry>
+          <material name="dark_gray"/>
+        </visual>
+      </xacro:unless>
+      <xacro:if value="$(arg box_visual)">
+        <xacro:box_visual xyz="0 0 -0.05" rpy="0 0 0" size="0.014 0.0285 0.114"/>
+      </xacro:if>
+      <xacro:box_collision xyz="0 0 -0.05" rpy="0 0 0" size="0.014 0.0285 0.114"/>
+      <xacro:box_inertial xyz="0 0 -0.05" rpy="0 0 0" size="0.014 0.0285 0.114" mass="0.0055"/>
+    </link>
+    <joint name="shin_r_rear_passive" type="revolute">
+      <parent link="thigh_r_middle_passive_link"/>
+      <child link="shin_r_rear_passive_link"/>
+      <origin xyz="0 0 -0.1" rpy="0 1.570796327 0"/>
+      <axis xyz="0 1 0"/>
+      <limit effort="0" lower="-1.570796327" upper="0.9948" velocity="1000.0"/>
+      <dynamics damping="0.0" friction="0.0"/>
+    </joint>
+    <link name="shin_r_rear_passive_link">
+      <xacro:unless value="$(arg box_visual)">
+        <visual>
+          <origin xyz="0 0 0" rpy="0 0 0"/>
+          <geometry>
+            <mesh filename="${MESH_DIR}/kuroko/stl/shin_r_rear_passive.stl"/>
+          </geometry>
+          <material name="dark_gray"/>
+        </visual>
+      </xacro:unless>
+      <xacro:if value="$(arg box_visual)">
+        <xacro:box_visual xyz="0 0 -0.05" rpy="0 0 0" size="0.014 0.0445 0.114"/>
+      </xacro:if>
+      <xacro:box_collision xyz="0 0 -0.05" rpy="0 0 0" size="0.014 0.0445 0.114"/>
+      <xacro:box_inertial xyz="0 0 -0.05" rpy="0 0 0" size="0.014 0.0445 0.114" mass="0.016"/>
+    </link>
+    <joint name="thigh_r_rear_passive_loop" type="revolute">
+      <parent link="shin_r_rear_passive_link"/>
+      <child link="thigh_r_rear_passive_lower_link"/>
+      <origin xyz="-0.00776457 0 -0.0289778" rpy="0 -1.570796327 0"/>
+      <axis xyz="0 1 0"/>
+      <limit effort="0" lower="-0.9948" upper="1.570796327" velocity="1000.0"/>
+      <dynamics damping="0.0" friction="0.0"/>
+    </joint>
+    <link name="thigh_r_rear_passive_lower_link">
+      <xacro:box_inertial xyz="0 0 0.05" rpy="0 0 0" size="0.014 0.0285 0.114" mass="0.0055"/>
+    </link>
+    <gazebo>
+      <plugin filename="libgz-sim-detachable-joint-system.so" name="gz::sim::systems::DetachableJoint">
+        <parent_link>thigh_r_rear_passive_upper_link</parent_link>
+        <child_model>${robot_name}</child_model>
+        <child_link>thigh_r_rear_passive_lower_link</child_link>
+      </plugin>
+    </gazebo>
+    <joint name="ankle_r_rear_passive" type="revolute">
+      <parent link="shin_r_rear_passive_link"/>
+      <child link="ankle_r_rear_passive_link"/>
+      <origin xyz="0 0 -0.1" rpy="0 -0.785398163 0"/>
+      <axis xyz="0 1 0"/>
+      <limit effort="0" lower="-0.4974" upper="1.8588" velocity="1000.0"/>
+      <dynamics damping="0.0" friction="0.0"/>
+      <mimic joint="shin_r_active" multiplier="-1" offset="0"/>
+    </joint>
+    <link name="ankle_r_rear_passive_link">
+      <xacro:unless value="$(arg box_visual)">
+        <visual>
+          <origin xyz="0.0335 0 0" rpy="0 0 0"/>
+          <geometry>
+            <mesh filename="${MESH_DIR}/kuroko/stl/ankle_r_pitch_passive.stl"/>
+          </geometry>
+          <material name="dark_gray"/>
+        </visual>
+      </xacro:unless>
+      <xacro:if value="$(arg box_visual)">
+        <xacro:box_visual xyz="0.005 0 -0.013" rpy="0 0 0" size="0.0855 0.0325 0.0465"/>
+      </xacro:if>
+      <xacro:box_collision xyz="0.005 0 -0.013" rpy="0 0 0" size="0.0855 0.0325 0.0465"/>
+      <xacro:box_inertial xyz="0.005 0 -0.013" rpy="0 0 0" size="0.0855 0.0325 0.0465"
+        mass="0.104"/>
+    </link>
+    <joint name="shin_r_front_passive_upper" type="revolute">
+      <parent link="knee_r_passive_link"/>
+      <child link="shin_r_front_passive_upper_link"/>
+      <origin xyz="0.0335 0 0" rpy="0 0.785398163 0"/>
+      <axis xyz="0 1 0"/>
+      <limit effort="0" lower="-1.570796327" upper="0.9948" velocity="1000.0"/>
+      <dynamics damping="0.0" friction="0.0"/>
+    </joint>
+    <link name="shin_r_front_passive_upper_link">
+      <xacro:unless value="$(arg box_visual)">
+        <visual>
+          <origin xyz="0 0 0" rpy="0 0 0"/>
+          <geometry>
+            <mesh filename="${MESH_DIR}/kuroko/stl/shin_r_front_passive.stl"/>
+          </geometry>
+          <material name="dark_gray"/>
+        </visual>
+      </xacro:unless>
+      <xacro:if value="$(arg box_visual)">
+        <xacro:box_visual xyz="0 0 -0.05" rpy="0 0 0" size="0.014 0.0445 0.114"/>
+      </xacro:if>
+      <xacro:box_collision xyz="0 0 -0.05" rpy="0 0 0" size="0.014 0.0385 0.114"/>
+      <xacro:box_inertial xyz="0 0 -0.05" rpy="0 0 0" size="0.014 0.0385 0.114" mass="0.0065"/>
+    </link>
+    <joint name="shin_r_front_passive_lower" type="revolute">
+      <parent link="ankle_r_rear_passive_link"/>
+      <child link="shin_r_front_passive_lower_link"/>
+      <origin xyz="0.0335 0 0" rpy="0 0.785398163 0"/>
+      <axis xyz="0 1 0"/>
+      <limit effort="0" lower="-1.570796327" upper="0.9948" velocity="1000.0"/>
+      <dynamics damping="0.0" friction="0.0"/>
+    </joint>
+    <link name="shin_r_front_passive_lower_link">
+      <xacro:box_inertial xyz="0 0 0.05" rpy="0 0 0" size="0.014 0.0385 0.114" mass="0.0065"/>
+    </link>
+    <gazebo>
+      <plugin filename="libgz-sim-detachable-joint-system.so" name="gz::sim::systems::DetachableJoint">
+        <parent_link>shin_r_front_passive_upper_link</parent_link>
+        <child_model>${robot_name}</child_model>
+        <child_link>shin_r_front_passive_lower_link</child_link>
+      </plugin>
+    </gazebo>
+    <joint name="ankle_r_roll" type="revolute">
+      <parent link="ankle_r_rear_passive_link"/>
+      <child link="ankle_r_roll_link"/>
+      <origin xyz="0.0185 0 -0.027" rpy="0 0 0"/>
+      <axis xyz="1 0 0"/>
+      <limit effort="3.1" lower="-0.3704" upper="1.5708" velocity="6.5"/>
+      <dynamics damping="0.477" friction="0.0"/>
+    </joint>
+    <link name="ankle_r_roll_link">
+      <xacro:unless value="$(arg box_visual)">
+        <visual>
+          <origin xyz="0 0 0" rpy="0 0 0"/>
+          <geometry>
+            <mesh filename="${MESH_DIR}/kuroko/stl/ankle_r_roll.stl"/>
+          </geometry>
+          <material name="dark_gray"/>
+        </visual>
+      </xacro:unless>
+      <xacro:if value="$(arg box_visual)">
+        <xacro:box_visual xyz="0 -0.009375 -0.01175" rpy="0 0 0" size="0.0365 0.05375 0.043"/>
+      </xacro:if>
+      <xacro:box_collision xyz="0 -0.009375 -0.01175" rpy="0 0 0" size="0.0365 0.05375 0.043"/>
+      <xacro:box_inertial xyz="0 -0.009375 -0.01175" rpy="0 0 0" size="0.0365 0.05375 0.043"
+        mass="0.136"/>
+    </link>
+    <joint name="ankle_r_yaw" type="revolute">
+      <parent link="ankle_r_roll_link"/>
+      <child link="ankle_r_yaw_link"/>
+      <origin xyz="0 0 -0.03825" rpy="0 0 0"/>
+      <axis xyz="0 0 1"/>
+      <limit effort="3.1" lower="-3.1" upper="3.1" velocity="6.5"/>
+      <dynamics damping="0.477" friction="0.0"/>
+    </joint>
+    <link name="ankle_r_yaw_link">
+      <xacro:unless value="$(arg box_visual)">
+        <visual>
+          <origin xyz="0 0 0" rpy="0 0 0"/>
+          <geometry>
+            <mesh filename="${MESH_DIR}/kuroko/stl/ankle_r_yaw.stl"/>
+          </geometry>
+          <material name="dark_gray"/>
+        </visual>
+      </xacro:unless>
+      <xacro:if value="$(arg box_visual)">
+        <xacro:box_visual xyz="0 0 -0.004" rpy="0 0 0" size="0.12 0.075 0.008"/>
+      </xacro:if>
+      <xacro:box_inertial xyz="0 0 -0.004" rpy="0 0 0" size="0.12 0.075 0.008" mass="0.043"/>
+      <!-- <xacro:box_collision xyz="0 0 -0.004" rpy="0 0 0" size="0.12 0.075 0.008"/> -->
+      <collision>
+        <origin xyz="0.052 0.0295 0" rpy="0 0 0"/>
+        <geometry>
+          <sphere radius="0.008"/>
+        </geometry>
+        <material name="gray"/>
+      </collision>
+      <collision>
+        <origin xyz="-0.052 0.0295 0" rpy="0 0 0"/>
+        <geometry>
+          <sphere radius="0.008"/>
+        </geometry>
+        <material name="gray"/>
+      </collision>
+      <collision>
+        <origin xyz="-0.052 -0.0295 0" rpy="0 0 0"/>
+        <geometry>
+          <sphere radius="0.008"/>
+        </geometry>
+        <material name="gray"/>
+      </collision>
+      <collision>
+        <origin xyz="0.052 -0.0295 0" rpy="0 0 0"/>
+        <geometry>
+          <sphere radius="0.008"/>
+        </geometry>
+        <material name="gray"/>
+      </collision>
+    </link>
   </xacro:macro>
 </robot>

Commit message: WIP

File: kuroko_description/xacro/kuroko/kuroko.xacro (robot description, xacro)
@@ -2,6 +2,7 @@
 <robot name="kuroko" xmlns:xacro="http://www.ros.org/wiki/xacro">
   <xacro:arg name="gazebo" default="false"/>
+  <xacro:arg name="gz_sim" default="false"/>
   <xacro:arg name="box_visual" default="false"/>
-  <xacro:arg name="gazebo_hw_interface" default="position"/>
+  <xacro:arg name="command_interface" default="position"/>
   <xacro:property name="XACRO_DIR" value="$(find kuroko_description)/xacro" />
   <xacro:property name="MESH_DIR" value="package://kuroko_description/meshes" />
@@ -28,5 +29,5 @@
   <!-- DOTO:Loading Gazebo Controllers for joints -->
   <!-- MACRO:Setting up a Robot Model -->
-  <xacro:macro name="kuroko_xacro" params="gazebo box_visual gazebo_hw_interface">
+  <xacro:macro name="kuroko_xacro" params="gazebo box_visual">
     <link name="body_link"/>
     <joint name="root_joint" type="fixed">
@@ -35,13 +36,13 @@
       <origin xyz="0 0 0" rpy="0 0 0"/>
     </joint>
-    <xacro:body_xacro box_visual="$(arg box_visual)"/>
+    <xacro:body_xacro box_visual="${box_visual}"/>
     <xacro:body_gazebo/>
-    <xacro:arm_r_xacro box_visual="$(arg box_visual)"/>
+    <xacro:arm_r_xacro box_visual="${box_visual}"/>
     <xacro:arm_r_gazebo/>
-    <xacro:arm_l_xacro box_visual="$(arg box_visual)"/>
+    <xacro:arm_l_xacro box_visual="${box_visual}"/>
     <xacro:arm_l_gazebo/>
-    <xacro:leg_r_xacro gazebo="$(arg gazebo)" box_visual="$(arg box_visual)"/>
+    <xacro:leg_r_xacro gazebo="${gazebo}" box_visual="${box_visual}"/>
     <xacro:leg_r_gazebo/>
-    <xacro:leg_l_xacro gazebo="$(arg gazebo)" box_visual="$(arg box_visual)"/>
+    <xacro:leg_l_xacro gazebo="${gazebo}" box_visual="${box_visual}"/>
     <xacro:leg_l_gazebo/>
     <xacro:imu_n100mini parent="waist_link" name="imu" namespace="/kuroko/sensors/imu">
@@ -60,5 +61,4 @@
   </xacro:macro>
   <!-- Load Macros -->
-  <xacro:kuroko_xacro gazebo="$(arg gazebo)" box_visual="$(arg box_visual)"
-    gazebo_hw_interface="$(arg gazebo_hw_interface)"/>
+  <xacro:kuroko_xacro gazebo="$(arg gazebo)" box_visual="$(arg box_visual)"/>
 </robot>
