Commit message: WIP

File: kuroko_description/xacro/kuroko/kuroko.xacro (robot description, xacro)
@@ -1,23 +1,39 @@
 <?xml version="1.0"?>
 <robot name="kuroko" xmlns:xacro="http://www.ros.org/wiki/xacro">
+  <!-- Arguments -->
   <xacro:arg name="gazebo" default="false"/>
   <xacro:arg name="gz_sim" default="false"/>
-  <xacro:arg name="command_interface" default="position"/>
   <xacro:arg name="box_visual" default="false"/>
-  <xacro:property name="XACRO_DIR" value="$(find kuroko_description)/xacro" />
-  <xacro:property name="MESH_DIR" value="package://kuroko_description/meshes" />
+  <!-- Controller selection -->
+  <xacro:arg name="controller" default="joint_trajectory_controller"/>
+  <!-- Optional explicit override; empty means infer from YAML (cmd_interfaces / interface_name / type defaults) -->
+  <xacro:arg name="command_interface" default=""/>
+  <!-- Semicolon-separated YAML list to be loaded by ros2_control plugin(s) -->
+  <xacro:arg name="controller_yaml_files"
+            default="$(find kuroko_description)/config/ros2_control/controller_manager.yaml;
+                      $(find kuroko_description)/config/ros2_control/joint_state_broadcaster.yaml;
+                      $(find kuroko_description)/config/ros2_control/joint_trajectory_controller.yaml"/>
+  <!-- Debug for xacro expansion -->
+  <xacro:arg name="debug_control" default="false"/>
+  <!-- Paths -->
+  <xacro:property name="XACRO_DIR" value="$(find kuroko_description)/xacro"/>
+  <xacro:property name="MESH_DIR" value="package://kuroko_description/meshes"/>
+  <!-- Includes: physics -->
   <xacro:include filename="${XACRO_DIR}/physics/materials.xacro"/>
   <xacro:include filename="${XACRO_DIR}/physics/box_physics.xacro"/>
   <xacro:include filename="${XACRO_DIR}/physics/gazebo_passive_joint.xacro"/>
+  <!-- Includes: parts -->
   <xacro:include filename="${XACRO_DIR}/kuroko/parts/body.xacro"/>
+  <xacro:include filename="${XACRO_DIR}/kuroko/parts/arm_r.xacro"/>
+  <xacro:include filename="${XACRO_DIR}/kuroko/parts/arm_l.xacro"/>
+  <xacro:include filename="${XACRO_DIR}/kuroko/parts/leg_r.xacro"/>
+  <xacro:include filename="${XACRO_DIR}/kuroko/parts/leg_l.xacro"/>
+  <!-- Includes: Gazebo Classic tags for each part -->
   <xacro:include filename="${XACRO_DIR}/kuroko/gazebo/body.gazebo"/>
-  <xacro:include filename="${XACRO_DIR}/kuroko/parts/arm_r.xacro"/>
   <xacro:include filename="${XACRO_DIR}/kuroko/gazebo/arm_r.gazebo"/>
-  <xacro:include filename="${XACRO_DIR}/kuroko/parts/arm_l.xacro"/>
   <xacro:include filename="${XACRO_DIR}/kuroko/gazebo/arm_l.gazebo"/>
-  <xacro:include filename="${XACRO_DIR}/kuroko/parts/leg_r.xacro"/>
   <xacro:include filename="${XACRO_DIR}/kuroko/gazebo/leg_r.gazebo"/>
-  <xacro:include filename="${XACRO_DIR}/kuroko/parts/leg_l.xacro"/>
   <xacro:include filename="${XACRO_DIR}/kuroko/gazebo/leg_l.gazebo"/>
+  <!-- Includes: sensors -->
   <xacro:include filename="${XACRO_DIR}/sensors/range/tfluna.xacro"/>
   <xacro:include filename="${XACRO_DIR}/sensors/imu/enable_gz_imu_plugin.xacro"/>
@@ -25,10 +41,19 @@
   <xacro:include filename="${XACRO_DIR}/sensors/camera/enable_gz_rendering_plugin.xacro"/>
   <xacro:include filename="${XACRO_DIR}/sensors/camera/usb_camera.xacro"/>
-  <!-- <xacro:include filename="${XACRO_DIR}/kuroko/gz/gz_sim_trajectory_control.xacro"/> -->
-  <!-- <xacro:include filename="${XACRO_DIR}/kuroko/gz/gz_sim_position_control.xacro"/> -->
+  <!-- ros2_control plugin macros -->
   <xacro:include filename="${XACRO_DIR}/gazebo/gazebo_ros2_control_plugin.xacro"/>
-  <!-- DOTO:Loading Gazebo Controllers for joints -->
-  <!-- MACRO:Setting up a Robot Model -->
-  <xacro:macro name="kuroko_xacro" params="gazebo box_visual">
+  <xacro:include filename="${XACRO_DIR}/gz/gz_ros2_control_plugin.xacro"/>
+  <!-- ====================================================================== -->
+  <!-- Macro: build the robot model                                            -->
+  <!-- ====================================================================== -->
+  <xacro:macro name="kuroko_model"
+               params="gazebo:=false
+                       gz_sim:=false
+                       box_visual:=false
+                       controller:=''
+                       controller_yaml_files:=''
+                       command_interface:=''
+                       debug_control:=false">
+    <!-- Base -->
     <link name="body_link"/>
     <joint name="root_joint" type="fixed">
@@ -37,14 +62,19 @@
       <origin xyz="0 0 0" rpy="0 0 0"/>
     </joint>
+    <!-- Body + limbs -->
     <xacro:body_xacro box_visual="${box_visual}"/>
-    <xacro:body_gazebo/>
     <xacro:arm_r_xacro box_visual="${box_visual}"/>
-    <xacro:arm_r_gazebo/>
     <xacro:arm_l_xacro box_visual="${box_visual}"/>
-    <xacro:arm_l_gazebo/>
     <xacro:leg_r_xacro gazebo="${gazebo}" box_visual="${box_visual}"/>
-    <xacro:leg_r_gazebo/>
     <xacro:leg_l_xacro gazebo="${gazebo}" box_visual="${box_visual}"/>
-    <xacro:leg_l_gazebo/>
+    <!-- Gazebo Classic visuals/physics tags for parts -->
+    <xacro:if value="${gazebo}">
+      <xacro:body_gazebo/>
+      <xacro:arm_r_gazebo/>
+      <xacro:arm_l_gazebo/>
+      <xacro:leg_r_gazebo/>
+      <xacro:leg_l_gazebo/>
+    </xacro:if>
+    <!-- Sensors -->
     <xacro:imu_n100mini parent="waist_link" name="imu" namespace="/kuroko/sensors/imu">
       <origin xyz="-0.04 0 -0.01" rpy="0 0 0"/>
@@ -56,10 +86,30 @@
       <origin xyz="0.07 0 -0.044" rpy="0 0 0"/>
     </xacro:tfluna>
-    <!-- <xacro:gz_sim_trajectory_control/> -->
-    <xacro:gz_sim_position_control/>
-    <xacro:enable_gz_rendering_plugin/>
-    <xacro:enable_gz_imu_plugin/>
+    <!-- Sensor plugins: Gazebo backends only -->
+    <xacro:if value="${gazebo or gz_sim}">
+      <xacro:enable_gz_rendering_plugin/>
+      <xacro:enable_gz_imu_plugin/>
+    </xacro:if>
+    <!-- ros2_control plugin injection -->
+    <!-- Gazebo Classic: expects gazebo_ros2_control_plugin macro to expand yaml_files -->
+    <xacro:gazebo_ros2_control_plugin
+      enabled="${gazebo}"
+      yaml_files="${controller_yaml_files}"/>
+    <!-- Gazebo Sim: use the new gz_ros2_control_setup macro -->
+    <xacro:gz_ros2_control_setup
+      enabled="${gz_sim}"
+      controller="${controller}"
+      yaml_files="${controller_yaml_files}"
+      command_interface="${command_interface}"
+      debug="${debug_control}"/>
   </xacro:macro>
-  <!-- Load Macros -->
-  <xacro:kuroko_xacro gazebo="$(arg gazebo)" box_visual="$(arg box_visual)"/>
+  <!-- Instantiate -->
+  <xacro:kuroko_model
+    gazebo="$(arg gazebo)"
+    gz_sim="$(arg gz_sim)"
+    box_visual="$(arg box_visual)"
+    controller="$(arg controller)"
+    controller_yaml_files="$(arg controller_yaml_files)"
+    command_interface="$(arg command_interface)"
+    debug_control="$(arg debug_control)"/>
 </robot>

Commit message: Set implicitSpringDamper

File: kuroko_description/xacro/kuroko/kuroko.xacro (robot description, xacro)
@@ -48,8 +48,8 @@
     <xacro:arm_l_xacro box_visual="${box_visual}"/>
     <xacro:arm_l_gazebo/>
-    <!-- <xacro:leg_r_xacro gazebo="${gazebo}" box_visual="${box_visual}"/>
+    <xacro:leg_r_xacro gazebo="${gazebo}" box_visual="${box_visual}"/>
     <xacro:leg_r_gazebo/>
     <xacro:leg_l_xacro gazebo="${gazebo}" box_visual="${box_visual}"/>
-    <xacro:leg_l_gazebo/> -->
+    <xacro:leg_l_gazebo/>
     <xacro:imu_n100mini parent="waist_link" name="imu" namespace="/kuroko/sensors/imu">
       <origin xyz="-0.04 0 -0.01" rpy="0 0 0"/>

File: kuroko_description/xacro/physics/default_gazebo_params.xacro (robot description, xacro)
@@ -19,3 +19,10 @@
     </gazebo>
   </xacro:macro>
+  <xacro:macro name="implicit_damping_joint" params="joint_name">
+    <gazebo reference="${joint_name}">
+      <implicitSpringDamper>1</implicitSpringDamper>
+      <stopCfm>1e-7</stopCfm>
+      <stopErp>0.8</stopErp>
+    </gazebo>
+  </xacro:macro>
 </robot>

Commit message: WIP

File: kuroko_description/xacro/kuroko/kuroko.xacro (robot description, xacro)
@@ -2,13 +2,5 @@
 <robot name="kuroko" xmlns:xacro="http://www.ros.org/wiki/xacro">
   <xacro:arg name="gazebo" default="false"/>
-  <xacro:arg name="gz_sim" default="false"/>
-  <!-- Which controller instance name you want to use (must match YAML) -->
-  <xacro:arg name="controller" default="joint_trajectory_controller"/>
-  <!-- Optional override; if empty, plugin macro may infer from YAML -->
-  <xacro:arg name="command_interface" default="position"/>
-  <!-- Single YAML file (absolute path recommended) -->
-  <xacro:arg name="controller_yaml" default=""/>
-  <!-- Print xacro-time debug messages -->
-  <xacro:arg name="debug_control" default="false"/>
+  <xacro:arg name="gazebo_hardware_interface" default="position"/>
   <xacro:arg name="box_visual" default="false"/>
   <xacro:property name="XACRO_DIR" value="$(find kuroko_description)/xacro" />
@@ -33,7 +25,7 @@
   <xacro:include filename="${XACRO_DIR}/sensors/camera/usb_camera.xacro"/>
   <!-- Gazebo Classic ros2_control helper -->
-  <xacro:include filename="${XACRO_DIR}/gazebo/gazebo_ros2_control_plugin.xacro"/>
+  <xacro:include filename="${XACRO_DIR}/kuroko/gazebo/kuroko_transmission.gazebo"/>
   <!-- Main robot model macro -->
-  <xacro:macro name="kuroko_model" params="gazebo box_visual">
+  <xacro:macro name="kuroko_model" params="gazebo gazebo_hardware_interface box_visual">
     <link name="body_link"/>
     <joint name="root_joint" type="fixed">
@@ -64,7 +56,14 @@
     <xacro:enable_gz_imu_plugin/>
     <!-- ros2_control (Gazebo Classic): enabled only when gazebo:=true -->
-    <xacro:gazebo_ros2_control_plugin controller_yaml="$(arg controller_yaml)"/>
+    <xacro:if value="${gazebo}">
+      <xacro:if value="${gazebo_hardware_interface=='position'}">
+        <xacro:kuroko_transmission_position/>
+      </xacro:if>
+      <xacro:if value="${gazebo_hardware_interface=='effort'}">
+        <xacro:kuroko_transmission_effort/>
+      </xacro:if>
+    </xacro:if>
   </xacro:macro>
   <!-- Instantiate -->
-  <xacro:kuroko_model gazebo="$(arg gazebo)" box_visual="$(arg box_visual)"/>
+  <xacro:kuroko_model gazebo="$(arg gazebo)" box_visual="$(arg box_visual)" gazebo_hardware_interface="$(arg gazebo_hardware_interface)"/>
 </robot>

Commit message: Fix bug

File: kuroko_description/xacro/kuroko/kuroko.xacro (robot description, xacro)
@@ -7,5 +7,10 @@
   <xacro:arg name="controller_yaml" default=""/>
   <xacro:property name="XACRO_DIR" value="$(find kuroko_description)/xacro" />
-  <xacro:property name="MESH_DIR" value="$(find kuroko_description)/meshes" />
+  <xacro:unless value="$(arg gazebo)">
+    <xacro:property name="MESH_DIR" value="package://kuroko_description/meshes" />
+  </xacro:unless>
+  <xacro:if value="$(arg gazebo)">
+    <xacro:property name="MESH_DIR" value="$(find kuroko_description)/meshes" />
+  </xacro:if>
   <xacro:include filename="${XACRO_DIR}/physics/materials.xacro"/>
   <xacro:include filename="${XACRO_DIR}/physics/box_physics.xacro"/>

Commit message: gazebo_hardware_interface -> gazebo_command_interface

File: kuroko_description/xacro/kuroko/kuroko.xacro (robot description, xacro)
@@ -2,5 +2,5 @@
 <robot name="kuroko" xmlns:xacro="http://www.ros.org/wiki/xacro">
   <xacro:arg name="gazebo" default="false"/>
-  <xacro:arg name="gazebo_hardware_interface" default="position"/>
+  <xacro:arg name="gazebo_command_interface" default="position"/>
   <xacro:arg name="box_visual" default="false"/>
   <!-- Optional ros2_control controller parameters YAML for Gazebo Classic plugin -->
@@ -34,5 +34,5 @@
   <xacro:include filename="${XACRO_DIR}/kuroko/gazebo/kuroko_command_interface.gazebo"/>
   <!-- Main robot model macro -->
-  <xacro:macro name="kuroko_model" params="gazebo gazebo_hardware_interface box_visual">
+  <xacro:macro name="kuroko_model" params="gazebo gazebo_command_interface box_visual">
     <link name="body_link"/>
     <joint name="root_joint" type="fixed">
@@ -63,12 +63,12 @@
     <xacro:enable_gz_imu_plugin/>
     <!-- ros2_control (Gazebo Classic): enabled only when gazebo:=true -->
-    <xacro:if value="${gazebo_hardware_interface=='position'}">
+    <xacro:if value="${gazebo_command_interface=='position'}">
       <xacro:kuroko_command_interface_position controller_yaml="$(arg controller_yaml)" />
     </xacro:if>
-    <xacro:if value="${gazebo_hardware_interface=='effort'}">
+    <xacro:if value="${gazebo_command_interface=='effort'}">
       <xacro:kuroko_command_interface_effort controller_yaml="$(arg controller_yaml)" />
     </xacro:if>
   </xacro:macro>
   <!-- Instantiate -->
-  <xacro:kuroko_model gazebo="$(arg gazebo)" box_visual="$(arg box_visual)" gazebo_hardware_interface="$(arg gazebo_hardware_interface)"/>
+  <xacro:kuroko_model gazebo="$(arg gazebo)" box_visual="$(arg box_visual)" gazebo_command_interface="$(arg gazebo_command_interface)"/>
 </robot>

Commit message: Read controllers from yaml

File: kuroko_description/xacro/kuroko/kuroko.xacro (robot description, xacro)
@@ -2,7 +2,7 @@
 <robot name="kuroko" xmlns:xacro="http://www.ros.org/wiki/xacro">
   <xacro:arg name="gazebo" default="false"/>
-  <xacro:arg name="gazebo_command_interface" default="position"/>
   <xacro:arg name="box_visual" default="false"/>
   <!-- Optional ros2_control controller parameters YAML for Gazebo Classic plugin -->
+  <!-- <xacro:arg name="controller_yaml" default="$(find kuroko_description)/config/ros2_control/joint_trajectory_controller.yaml"/> -->
   <xacro:arg name="controller_yaml" default="$(find kuroko_description)/config/ros2_control/joint_trajectory_controller.yaml"/>
   <xacro:arg name="pid_yaml" default="$(find kuroko_description)/config/ros2_control/gazebo_pid_gains.yaml"/>
@@ -35,5 +35,5 @@
   <xacro:include filename="${XACRO_DIR}/kuroko/gazebo/kuroko_command_interface.gazebo"/>
   <!-- Main robot model macro -->
-  <xacro:macro name="kuroko_model" params="gazebo gazebo_command_interface box_visual">
+  <xacro:macro name="kuroko_model" params="gazebo box_visual">
     <link name="body_link"/>
     <joint name="root_joint" type="fixed">
@@ -71,4 +71,4 @@
   </xacro:macro>
   <!-- Instantiate -->
-  <xacro:kuroko_model gazebo="$(arg gazebo)" box_visual="$(arg box_visual)" gazebo_command_interface="$(arg gazebo_command_interface)"/>
+  <xacro:kuroko_model gazebo="$(arg gazebo)" box_visual="$(arg box_visual)"/>
 </robot>

Commit message: WIP

File: kuroko_description/xacro/kuroko/kuroko.xacro (robot description, xacro)
@@ -52,7 +52,7 @@
     <xacro:leg_l_xacro gazebo="${gazebo}" box_visual="${box_visual}"/>
     <xacro:leg_l_gazebo/>
-    <!-- <xacro:imu_n100mini parent="waist_link" name="imu" namespace="/kuroko/sensors/imu">
+    <xacro:imu_n100mini parent="waist_link" name="imu" namespace="/kuroko/sensors/imu">
       <origin xyz="-0.04 0 -0.01" rpy="0 0 0"/>
-    </xacro:imu_n100mini> -->
+    </xacro:imu_n100mini>
     <!-- <xacro:usb_camera parent="waist_link" name="camera" namespace="/kuroko/sensors/camera">
       <origin xyz="0.07 0 -0.026" rpy="0 0 0"/>

File: kuroko_description/xacro/sensors/imu/enable_gz_imu_plugin.xacro (robot description, xacro)
@@ -2,5 +2,5 @@
 <robot xmlns:xacro="http://www.ros.org/wiki/xacro">
   <xacro:macro name="enable_gz_imu_plugin">
-    <!-- Loading Gazebo Plugin for IMU -->
+    <!-- Loading gz Plugin for IMU -->
     <gazebo>
       <plugin name="gz::sim::systems::Imu" filename="gz-sim-imu-system"/>

File: kuroko_description/xacro/sensors/imu/imu_n100mini.xacro (robot description, xacro)
@@ -1,5 +1,5 @@
 <?xml version="1.0" encoding="UTF-8"?>
 <robot xmlns:xacro="http://www.ros.org/wiki/xacro">
-  <xacro:include filename="imu_n100mini_gazebo.xacro"/>
+  <xacro:include filename="imu_n100mini_gz.xacro"/>
   <xacro:macro name="imu_n100mini" params="name parent:='base_link' update_rate:=400 *origin namespace">
     <xacro:property name="depth" value="0.01"/>
@@ -34,5 +34,5 @@
       <preserveFixedJoint>true</preserveFixedJoint>
     </gazebo>
-    <xacro:n100mini_gazebo name="${name}" update_rate="${update_rate}" namespace="${namespace}"/>
+    <xacro:n100mini_gz name="${name}" update_rate="${update_rate}" namespace="${namespace}"/>
   </xacro:macro>
 </robot>

File: kuroko_description/xacro/sensors/imu/imu_n100mini_gz.xacro (robot description, xacro)
@@ -1,5 +1,5 @@
 <?xml version="1.0" encoding="UTF-8"?>
 <robot xmlns:xacro="http://www.ros.org/wiki/xacro">
-  <xacro:macro name="n100mini_gazebo" params="namespace name update_rate">
+  <xacro:macro name="n100mini_gz" params="namespace name update_rate">
     <gazebo reference="${name}_link">
       <material>Gazebo/Gray</material>

Commit message: WIP

File: kuroko_description/xacro/kuroko/kuroko.xacro (robot description, xacro)
@@ -28,7 +28,8 @@
   <xacro:include filename="${XACRO_DIR}/kuroko/gazebo/leg_l.gazebo"/>
   <xacro:include filename="${XACRO_DIR}/sensors/range/tfluna.xacro"/>
-  <xacro:include filename="${XACRO_DIR}/sensors/imu/enable_gz_imu_plugin.xacro"/>
+  <!-- <xacro:include filename="${XACRO_DIR}/sensors/imu/enable_gz_imu_plugin.xacro"/> -->
   <xacro:include filename="${XACRO_DIR}/sensors/imu/imu_n100mini.xacro"/>
-  <xacro:include filename="${XACRO_DIR}/sensors/camera/enable_gz_rendering_plugin.xacro"/>
+  <xacro:include filename="${XACRO_DIR}/sensors/imu/imu_n100mini_gazebo.xacro"/>
+  <!-- <xacro:include filename="${XACRO_DIR}/sensors/camera/enable_gz_rendering_plugin.xacro"/> -->
   <xacro:include filename="${XACRO_DIR}/sensors/camera/usb_camera.xacro"/>
   <!-- Gazebo Classic ros2_control helper -->
@@ -52,7 +53,8 @@
     <xacro:leg_l_xacro gazebo="${gazebo}" box_visual="${box_visual}"/>
     <xacro:leg_l_gazebo/>
-    <xacro:imu_n100mini parent="waist_link" name="imu" namespace="/kuroko/sensors/imu">
+    <xacro:imu_n100mini parent="waist_link" name="imu">
       <origin xyz="-0.04 0 -0.01" rpy="0 0 0"/>
     </xacro:imu_n100mini>
+    <xacro:n100mini_gazebo name="imu" namespace="/kuroko/sensors/imu"/>
     <!-- <xacro:usb_camera parent="waist_link" name="camera" namespace="/kuroko/sensors/camera">
       <origin xyz="0.07 0 -0.026" rpy="0 0 0"/>
@@ -61,5 +63,5 @@
       <origin xyz="0.07 0 -0.044" rpy="0 0 0"/>
     </xacro:tfluna> -->
-    <!-- Gazebo-specific sensor/plugins only when gazebo:=true -->
+    <!-- gz sensor/plugins -->
     <!-- <xacro:if value="${gazebo}">
       <xacro:enable_gz_rendering_plugin/>

File: kuroko_description/xacro/sensors/imu/imu_n100mini.xacro (robot description, xacro)
@@ -1,6 +1,5 @@
 <?xml version="1.0" encoding="UTF-8"?>
 <robot xmlns:xacro="http://www.ros.org/wiki/xacro">
-  <xacro:include filename="imu_n100mini_gz.xacro"/>
-  <xacro:macro name="imu_n100mini" params="name parent:='base_link' update_rate:=400 *origin namespace">
+  <xacro:macro name="imu_n100mini" params="name parent:='base_link' *origin">
     <xacro:property name="depth" value="0.01"/>
     <xacro:property name="width" value="0.01"/>
@@ -34,5 +33,4 @@
       <preserveFixedJoint>true</preserveFixedJoint>
     </gazebo>
-    <xacro:n100mini_gz name="${name}" update_rate="${update_rate}" namespace="${namespace}"/>
   </xacro:macro>
 </robot>

File: kuroko_description/xacro/sensors/imu/imu_n100mini_gz.xacro (robot description, xacro)
@@ -10,10 +10,4 @@
         <gz_frame_id>${name}_link</gz_frame_id>
       </sensor>
-      <sensor name="magnetometer" type="magnetometer">
-        <always_on>true</always_on>
-        <update_rate>${update_rate}</update_rate>
-        <topic>${namespace}/mag</topic>
-        <gz_frame_id>${name}_link</gz_frame_id>
-      </sensor>
     </gazebo>
   </xacro:macro>
